File: BreadBoard/LCD_Driver.kicad_sch (KiCad schematic)
At the start: 55 parts

Commit message: work on lcd driver
Parts:
- removed C? (x2): 1uF, Adafruit RA8875 TFT Breakout:0805-NO, symbol Adafruit RA8875 TFT Breakout-eagle-import:CAP_CERAMIC0805-NOOUTLINE
- removed C?: 0.1uF, Adafruit RA8875 TFT Breakout:0603-NO, symbol Adafruit RA8875 TFT Breakout-eagle-import:CAP_CERAMIC0603_NO
- removed C?: 10uF, Adafruit RA8875 TFT Breakout:0805-NO, symbol Adafruit RA8875 TFT Breakout-eagle-import:CAP_CERAMIC0805-NOOUTLINE
- removed D?: MBR0540, Adafruit RA8875 TFT Breakout:SOD-123, symbol Adafruit RA8875 TFT Breakout-eagle-import:DIODESOD-123
- removed D? (x2): 1N4148, Adafruit RA8875 TFT Breakout:SOD-323_MINI, symbol Adafruit RA8875 TFT Breakout-eagle-import:DIODE_SOD323MINI
- removed L?: 6.8uH large inductor, Adafruit RA8875 TFT Breakout:INDUCTOR_5X5MM_NR5040_NOTHERMALS, symbol Adafruit RA8875 TFT Breakout-eagle-import:INDUCTORNR5040
- removed R?: 2Ω, Adafruit RA8875 TFT Breakout:0805-NO, symbol Adafruit RA8875 TFT Breakout-eagle-import:RESISTOR0805_NOOUTLINE
- removed R? (x2): 8.2Ω, Adafruit RA8875 TFT Breakout:0805-NO, symbol Adafruit RA8875 TFT Breakout-eagle-import:RESISTOR0805_NOOUTLINE
- removed R?: 10K, Adafruit RA8875 TFT Breakout:0603-NO, symbol Adafruit RA8875 TFT Breakout-eagle-import:RESISTOR_0603_NOOUT
- removed SJ?: +25mA, Adafruit RA8875 TFT Breakout:SOLDERJUMPER_ARROW_NOPASTE, symbol Adafruit RA8875 TFT Breakout-eagle-import:SOLDERJUMPER
- removed SJ?: +100mA, Adafruit RA8875 TFT Breakout:SOLDERJUMPER_ARROW_NOPASTE, symbol Adafruit RA8875 TFT Breakout-eagle-import:SOLDERJUMPER
- removed U?: TPS61169, Adafruit RA8875 TFT Breakout:SC70-5, symbol Adafruit RA8875 TFT Breakout-eagle-import:VREG_BOOST_5PIN_SC70
- added C13, C14, C15: C, symbol Device:C
- added D1: MBR0540, Diode_SMD:D_SOD-123, symbol Diode:MBR0540
- added L1: L, symbol Device:L
- added R1: R, symbol Device:R
- added U2: TPS61165DRV, Package_SON:WSON-6-1EP_2x2mm_P0.65mm_EP1x1.6mm, symbol Driver_LED:TPS61165DRV
- gave numbers to parts that had none: 24
Connections:
- net +3V3: now also IC2.5 (VCC)
- net B3: now also R4.5 (2); no longer R4.8 (2)
- net B4: now also R4.6 (2); no longer R4.8 (2)
- net B5: now also R4.7 (2); no longer R4.8 (2)
- net B7: now also R5.5 (2); no longer R5.8 (2)
- net G2: now also R5.6 (2); no longer R5.8 (2)
- net G3: now also R5.7 (2); no longer R5.8 (2)
- net G5: now also R6.5 (2); no longer R6.8 (2)
- net G6: now also R6.6 (2); no longer R6.8 (2)
- net G7: now also R6.7 (2); no longer R6.8 (2)
- net GND: now also IC2.3 (GND), C13.2, C14.2, C15.2, R1.2, U2.3 (GND), U2.7 (GND)
- net HSYNC: now also R8.5 (2); no longer R8.8 (2)
- net MISO: no longer IC2.4 (O)
- net PIXCLK: now also R8.7 (2); no longer R8.8 (2)
- net R4: now also R7.5 (2); no longer R7.8 (2)
- net R5: now also R7.6 (2); no longer R7.8 (2)
- net R6: now also R7.7 (2); no longer R7.8 (2)
- net VSYNC: now also R8.6 (2); no longer R8.8 (2)
- net at U1.59 (PDAT8): now also R6.4 (1); no longer R6.1
- net at U1.47 (HSYNC): now also R8.4 (1); no longer R8.1
- net at U1.48 (VSYNC): now also R8.3 (1); no longer R8.1
- net at U1.49 (PCLK): now also R8.2 (1); no longer R8.1
- net at U1.51 (PDAT0): now also R4.4 (1); no longer R4.1
- net at U1.52 (PDAT1): now also R4.3 (1); no longer R4.1
- net at U1.53 (PDAT2): now also R4.2 (1); no longer R4.1
- net at U1.55 (PDAT4): now also R5.4 (1); no longer R5.1
- net at U1.56 (PDAT5): now also R5.3 (1); no longer R5.1
- net at U1.57 (PDAT6): now also R5.2 (1); no longer R5.1
- net at U1.63 (PDAT9): now also R6.3 (1); no longer R6.1
- net at U1.64 (PDAT10): now also R6.2 (1); no longer R6.1
- net at U1.66 (PDAT12): now also R7.4 (1); no longer R7.1
- net at U1.67 (PDAT13): now also R7.3 (1); no longer R7.1
- net at U1.68 (PDAT14): now also R7.2 (1); no longer R7.1
- new net: C15.1, D1.1 (K), R1.1, U2.1 (FB)
- new net: D1.2 (A), L1.2, U2.4 (SW)
- new net: C14.1, U2.2 (COMP)
- new net 12V: C13.1, L1.1, U2.6 (VIN)
- no-connect marks 1 -> 2
Other:
- note removed: "7 x 3.2V LED boost"

Commit message: update
Parts:
- removed C10, C11, C12, C5, C6, C7, C8, C9: 0.1uF, Adafruit RA8875 TFT Breakout:0603-NO, symbol Adafruit RA8875 TFT Breakout-eagle-import:CAP_CERAMIC0603_NO
- removed C14: C, symbol Device:C
- removed C4: 1uF, Adafruit RA8875 TFT Breakout:0805-NO, symbol Adafruit RA8875 TFT Breakout-eagle-import:CAP_CERAMIC0805-NOOUTLINE
- removed R12: 10K, Adafruit RA8875 TFT Breakout:0603-NO, symbol Adafruit RA8875 TFT Breakout-eagle-import:RESISTOR_0603_NOOUT
- removed U2: TPS61165DRV, Package_SON:WSON-6-1EP_2x2mm_P0.65mm_EP1x1.6mm, symbol Driver_LED:TPS61165DRV
- removed U5: 74HC4050, Adafruit RA8875 TFT Breakout:TSSOP16, symbol Adafruit RA8875 TFT Breakout-eagle-import:74HC4050DTSSOP
- added C1, C10, C3, C4, C5, C6, C7, C8, C9: 0.1uF, symbol Device:C
- added C2: 1uF, symbol Device:C
- added D1, D3: 1N4148, Diode_THT:D_DO-35_SOD27_P7.62mm_Horizontal, symbol Diode:1N4148
- added R2: 2Ω, symbol Device:R
- added R3, R4: 10k, symbol Device:R
- added U1: TPS61169DCKR, TPS61169DCKR:SOT65P210X110-5N, symbol TPS61169DCKR:TPS61169DCKR
- added U2: 74HC4050, Adafruit RA8875 TFT Breakout:SOIC16, symbol Adafruit RA8875 TFT Breakout-eagle-import:74HC4050D
- C16: renamed from C13; value C -> 10uF
- C?: renamed from C15; value C -> 1uF
- R?: renamed from R1; value R -> 8.2Ω
- renumbered L1 to 6.8uH, C3 to C?, C1 to C?, C2 to C?, D1 to D2, IC2 to IC?, J2 to J?, R6 to R?, R7 to R?, R5 to R?, R4 to R?, R8 to R?, R3 to R?, U1 to U?, Y1 to Y?
Connections:
- net 12V is gone; now on net VIN: 6.8uH.1, C16.1
- net +3V3: no longer IC?.5 (VCC)
- net B3: now also R?.8 (2); no longer R?.5 (2)
- net B4: now also R?.8 (2); no longer R?.6 (2)
- net B5: now also R?.8 (2); no longer R?.7 (2)
- net B7: now also R?.8 (2); no longer R?.5 (2)
- net CS: now also U2.7 (3A)
- net G2: now also R?.8 (2); no longer R?.6 (2)
- net G3: now also R?.8 (2); no longer R?.7 (2)
- net G5: now also R?.8 (2); no longer R?.5 (2)
- net G6: now also R?.8 (2); no longer R?.6 (2)
- net G7: now also R?.8 (2); no longer R?.7 (2)
- net GND: now also C1.2, C10.2, C2.2, C3.2, C4.2, C5.2, C6.2, C7.2, C8.2, C9.2, R2.2, U1.2 (GND), U2.8 (GND); no longer IC?.3 (GND)
- net HSYNC: now also R?.8 (2); no longer R?.5 (2)
- net MISO: now also IC?.4 (O)
- net MOSI: now also U2.5 (2A)
- net MOSI_3V: now also U2.4 (2Y)
- net PIXCLK: now also R?.8 (2); no longer R?.7 (2)
- net R4: now also R?.8 (2); no longer R?.5 (2)
- net R5: now also R?.8 (2); no longer R?.6 (2)
- net R6: now also R?.8 (2); no longer R?.7 (2)
- net RESET: now also R4.2, U2.9 (4A)
- net RESET_3V: now also U2.10 (4Y)
- net SCK: now also U2.3 (1A)
- net SPI_CLK_3V: now also U2.2 (1Y)
- net SPI_CS_3V: now also U2.6 (3Y)
- net VIN: now also R3.1, U1.5 (VIN)
- net VSYNC: now also R?.8 (2); no longer R?.6 (2)
- net at U?.59 (PDAT8): now also R?.1; no longer R?.4 (1)
- net at C?.1, D2.1 (K): no longer R?.1
- net at U?.47 (HSYNC): now also R?.1; no longer R?.4 (1)
- net at U?.48 (VSYNC): now also R?.1; no longer R?.3 (1)
- net at U?.49 (PCLK): now also R?.1; no longer R?.2 (1)
- net at U?.51 (PDAT0): now also R?.1; no longer R?.4 (1)
- net at U?.52 (PDAT1): now also R?.1; no longer R?.3 (1)
- net at U?.53 (PDAT2): now also R?.1; no longer R?.2 (1)
- net at U?.55 (PDAT4): now also R?.1; no longer R?.4 (1)
- net at U?.56 (PDAT5): now also R?.1; no longer R?.3 (1)
- net at U?.57 (PDAT6): now also R?.1; no longer R?.2 (1)
- net at U?.63 (PDAT9): now also R?.1; no longer R?.3 (1)
- net at U?.64 (PDAT10): now also R?.1; no longer R?.2 (1)
- net at U?.66 (PDAT12): now also R?.1; no longer R?.4 (1)
- net at U?.67 (PDAT13): now also R?.1; no longer R?.3 (1)
- net at U?.68 (PDAT14): now also R?.1; no longer R?.2 (1)
- net at 6.8uH.2, D2.2 (A): now also U1.1 (SW)
- new net: D1.2 (A), D3.2 (A), R3.2, U1.4 (CTRL)
- new net +1.5V: C10.1, C7.1, C8.1, C9.1
- new net +3.3V: C2.1, C3.1, C4.1, C5.1, C6.1, R4.1, U2.1 (VCC)
- new net LEDK: C1.1, R2.1, R?.1, U1.3 (FB)
Other:
- moved on the sheet: 6.8uH, C15, C16, D2, R1
