File: BreadBoard_git/BreadBoard_git.kicad_sch (KiCad schematic)
At the start: 41 parts, among them J1 24V DC wall plug-iN, J2 LCD Driver, Q1 CSD18512Q5B, Q2 CSD18512Q5B, Q3 RQ3E110AJTB, Q4 RQ3E110AJTB, Q5 RQ3E110AJTB, U1 ESP32-S3, U2 LM73605RNPR, U3 LM5148RGYR, U4 SHT45

Commit message: potential poverwrite
Parts:
- removed C1: APXE6R3ARA101ME61G, CHEMI-E61, symbol cout:APXE6R3ARA101ME61G
- removed C3, C9: GRM155R71A104KA01D, GRM155R71A104KA01D:CAPC1005X55N, symbol cboot:GRM155R71A104KA01D
- removed C4: CL05C821JB5NNNC, CL05C821JB5NNNC:CAPC1005X55N, symbol ccomp:CL05C821JB5NNNC
- removed C5: C0402C300J5GACTU, CAPC10555_55N_KEM, symbol ccomp2:C0402C300J5GACTU
- removed C6: C2012X6S1H155K125AB, C2012X6S1H155K125AB:CAPC2012X145N, symbol cin:C2012X6S1H155K125AB
- removed C7: MSAST21GBB5106MTNA01, MSAST21GBB5106MTNA01:CAPC2012X145N, symbol cout2:MSAST21GBB5106MTNA01
- removed C8: GRM188R71A225KE15D, G-188_MUR, symbol cvcc:GRM188R71A225KE15D
- removed Cff1: 16pF, symbol Device:C
- removed Coutx2: 470nF, symbol Device:C
- removed L2: 3.9uH, symbol Device:L
- removed L3: CDEP63MENP-R68MC, IND_CDEP63MENP-R68MC_SUM, symbol l1:CDEP63MENP-R68MC
- removed Rfbb1: 43.2kOhm, symbol Device:R
- removed Rfbt1: 100kOhm, symbol Device:R
- removed Rpgood1: 105kOhm, symbol Device:R
- added C1: C1608X6S1H474K080AB, C1608X6S1H474K080AB:CAPC1608X90N, symbol coutx:C1608X6S1H474K080AB
- added C3: GRM1555C1H160JA01D, GRM1555C1H160JA01D:CAPC1005X55N, symbol cff:GRM1555C1H160JA01D
- added Cboot2, Cvdda1: 100nF, symbol Device:C
- added Ccomp1: 820.0pF, symbol Device:C
- added Ccomp2: 30.0pF, symbol Device:C
- added Cin1: 1.5uF, symbol Device:C
- added Cout1: 10uF, symbol Device:C
- added Cvcc2: 2.2uF, symbol Device:C
- added L1: 680nH, symbol Device:L
- added L3: SRU8043-3R9Y, SRU80433R9Y, symbol L1:SRU8043-3R9Y
- added R1: CRCW040243K2FKED, CRCW040243K2FKED:RESC1005X40N, symbol Rfbb:CRCW040243K2FKED
- added R2: CRCW0402100KFKED, CRCW0402100KFKED:RESC1005X40N, symbol rfbt:CRCW0402100KFKED
- added R3: RC0201FR-07105KL, RC0201FR-07105KL:RESC0603X26N, symbol rpgood:RC0201FR-07105KL
- renumbered Rcomp to Rcomp1, Rconfig to Rconfig1, Rpg to Rpg1, Rsense to Rsense1, Rt to Rt1, Rvdda to Rvdda1, Vin to Vin1
Connections:
- net 3.3V: now also C1.2, C3.2, L3.2, R2.2, R3.2
- net DAP: now also C1.1, Cin1.2, Cvcc2.2, Cvdda1.2, R1.1
- net GNDREF: now also Cout1.2
- net Heater Vcc: now also Cout1.1
- net at U2.11 (FB): now also C3.1, R1.2, R2.1
- net at Rcomp1.1: now also Ccomp1.2
- net at Rcomp1.2, U3.5 (EXTCOMP): now also Ccomp2.2
- net at Q1.1, Q1.2, Q1.3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: now also Cboot2.2, L1.1
- net at Q1.5_8, U3.12 (VIN), U3.19 (EN)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: now also Cin1.1
- net at Cboot1.2, U2.1 (SW_1), U2.2 (SW_2)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: now also L3.1
- net at Rpg1.1, U3.9 (VCC): now also Cvcc2.1
- net at U3.15 (CBOOT): now also Cboot2.1
- net at Rvdda1.2, U3.18 (PFM/SYNC), U3.8 (VDDA): now also Cvdda1.1
- net at Rsense1.1, U3.20 (ISNS+): now also L1.2
- net at U2.16 (PGOOD): now also R3.1
- new net: Ccomp1.1, Ccomp2.1
Other:
- moved on the sheet: Rsense1

Commit message: footprints not working
Parts:
- removed Cboot1: 470nF, symbol Device:C
- removed Cboot2, Cvdda1: 100nF, symbol Device:C
- removed Cbulk1: 100uF, symbol Device:C_US
- removed Ccomp1: 820.0pF, symbol Device:C
- removed Ccomp2: 30.0pF, symbol Device:C
- removed Cin1: 1.5uF, symbol Device:C
- removed Cin2: 10uF (2), symbol Device:C
- removed Cinx2: 47nF, symbol Device:C
- removed Cout1: 10uF, symbol Device:C
- removed Cvcc1, Cvcc2: 2.2uF, symbol Device:C
- removed L1: 680nH, symbol Device:L
- removed Rcomp1: 4.87kOhm, symbol Device:R
- removed Rconfig1: 40.2kOhm, symbol Device:R
- removed Rpg1: 100kOmh, symbol Device:R
- removed Rsense1: 3.0Ohm, symbol Device:R
- removed Rt1: 9.53kOhm, symbol Device:R
- removed Rvdda1: 47.5kOmh, symbol Device:R
- added C10: GRM155R71A104KA01D, GRM155R71A104KA01D:CAPC1005X55N, symbol cboot_5:GRM155R71A104KA01D
- added C11: GRM155R60J474KE19D, G-155_MUR, symbol cboot:GRM155R60J474KE19D
- added C12: CL05C821JB5NNNC, CL05C821JB5NNNC:CAPC1005X55N, symbol ccomp_5:CL05C821JB5NNNC
- added C13: C0402C300J5GACTU, CAPC10555_55N_KEM, symbol ccomp2_5:C0402C300J5GACTU
- added C14: GRM188R71A225KE15D, G-188_MUR, symbol cvcc_5:GRM188R71A225KE15D
- added C15: GRM155R71A104KA01D, GRM155R71A104KA01D:CAPC1005X55N, symbol cvdda_5:GRM155R71A104KA01D
- added C16, C17, C18, C19: C2012X6S1H155K125AB, C2012X6S1H155K125AB:CAPC2012X145N, symbol cin_5:C2012X6S1H155K125AB
- added C20, C21, C22, C9: MSAST21GBB5106MTNA01, MSAST21GBB5106MTNA01:CAPC2012X145N, symbol cout_5:MSAST21GBB5106MTNA01
- added C4: GRM21BR71A225KA01L, CAP_GRM21_MUR, symbol cvcc:GRM21BR71A225KA01L
- added C5: C1005X7R1H473K050BB, CAP_1005_TDK, symbol cinx:C1005X7R1H473K050BB
- added C6, C8: CL32A106KBJNNNE, CL32A106KBJNNNE:CAPC3225X270N, symbol cin:CL32A106KBJNNNE
- added C7: UUD1V101MNL1GS, U2-P_NCH, symbol cbulk:UUD1V101MNL1GS
- added IC1: IAUCN04S7L028ATMA1, IAUC120N06S5N011ATMA1, symbol M1_5:IAUCN04S7L028ATMA1
- added L2: CDEP63MENP-R68MC, IND_CDEP63MENP-R68MC_SUM, symbol L1_5:CDEP63MENP-R68MC
- added R4: WSR23L000FEA, WSR, symbol rsense_5:WSR23L000FEA
- added R5: RC0603FR-079K53L, RC0603N_YAG, symbol rt_5:RC0603FR-079K53L
- added R6: RC0603FR-0740K2L, RC0603N_YAG, symbol rconfig_5:RC0603FR-0740K2L
- added R7: CRCW04024K87FKED, RES_CRCW_0402, symbol rcomp_5:CRCW04024K87FKED
- added R8: CRCW0603100KFKEA, CRCW0603100KFKEA:RESC1508X50N, symbol rpg_5:CRCW0603100KFKEA
- added R9: CRCW060347K5FKEA, RES_CRCW_0603, symbol rvdda_5:CRCW060347K5FKEA
- added U5: CSD17577Q5A, DQJ8, symbol M2_5:CSD17577Q5A
- F1: footprint (none) -> Resistor_SMD:R_2512_6332Metric
- J1: footprint (none) -> Connector_BarrelJack:BarrelJack_Horizontal
Connections:
- net Heater Vcc is gone; now on net GNDREF: U3.21 (VOUT)
- net DAP: now also C14.1, C15.1, C16.1, C17.1, C18.1, C19.1, C4.1, C5.1, C6.1, C7.2, C8.1, R5.2, R6.2
- net GNDREF: now also C20.1, C20.2, C21.1, C21.2, C22.1, C22.2, C9.1, C9.2, R4.2
- net at U3.5 (EXTCOMP): now also C13.2, R7.1
- net at U2.18 (EN), U2.20 (PVIN_20), U2.21 (PVIN_21)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: now also C5.2, C6.2, C7.1, C8.2
- net at Q1.1, Q1.2, Q1.3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: now also C10.1, L2.2
- net at U3.20 (ISNS+): now also L2.1, R4.1
- net at U3.9 (VCC): now also C14.2, R8.2
- net at U2.7 (VCC): now also C4.2
- net at Q1.5_8, U3.12 (VIN), U3.19 (EN)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: now also C16.2, C17.2, C18.2, C19.2
- net at U2.6 (CBOOT): now also C11.1
- net at L3.1, U2.1 (SW_1), U2.2 (SW_2)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: now also C11.2
- net at U3.6 (FB): now also R9.2
- net at U3.18 (PFM/SYNC), U3.8 (VDDA): now also C15.2, R9.1
- net at U3.15 (CBOOT): now also C10.2
- net at U3.3 (CNFG): now also R6.1
- net at U3.17 (PG/SYNCOUT): now also R8.1
- net at U3.4 (RT): now also R5.1
- new net: C12.1, C13.1
- new net: C12.2, R7.2
Other:
- note added: "12V Buck"
- note added: "SCREW TERMINALS"
- note added: "SDA AND SCL WILL BE JUMPER WIRES"
- moved on the sheet: Vin1

Commit message: small updates
Parts:
- added J3: Conn_01x15_Socket, symbol Connector:Conn_01x15_Socket
- added U6: ESP32-S3-WROOM-1, RF_Module:ESP32-S3-WROOM-1, symbol RF_Module:ESP32-S3-WROOM-1
Connections:
- net +3.3V: now also J3.1 (Pin_1)
- net DAP: now also J3.2 (Pin_2), U6.1 (GND), U6.40 (GND), U6.41 (GND)
- net DRIVER_CS: no longer U1.15 (GPIO10)
- net DRIVER_INT: no longer U1.27 (GPIO21)
- net DRIVER_MISO: no longer U1.18 (GPIO13)
- net DRIVER_MOSI: no longer U1.16 (GPIO11)
- net DRIVER_RST: no longer U1.14 (GPIO9)
- net DRIVER_SCK: no longer U1.17 (GPIO12)
- new net: J3.9 (Pin_9), U1.14 (GPIO9)
- new net: J3.8 (Pin_8), U1.15 (GPIO10)
- new net: J3.7 (Pin_7), U1.16 (GPIO11)
- new net: J3.5 (Pin_5), U1.17 (GPIO12)
- new net: J3.6 (Pin_6), U1.18 (GPIO13)
- new net: J3.11 (Pin_11), U1.27 (GPIO21)
- no-connect marks 46 -> 53
