File: BreadBoard_git/BreadBoard_git.kicad_sch (KiCad schematic)
At the start: 63 parts, among them IC1 IAUCN04S7L028ATMA1, J1 24V DC wall plug-iN, J2 Conn_01x05_Socket, J3 Conn_01x15_Socket, J4 USB4105-GF-A, Q1 CSD18512Q5B, Q2 CSD18512Q5B, Q3 RQ3E110AJTB, Q4 RQ3E110AJTB, Q5 RQ3E110AJTB, SW1 SW_DPST_x2, SW2 SW_DPST_x2, U2 LM73605RNPR, U3 LM5148RGYR, U5 CSD17577Q5A, U6 ESP32-S3-WROOM-1

Commit message: updated
Parts:
- removed C1: C1608X6S1H474K080AB, CAP_1608_TDK, symbol coutx:C1608X6S1H474K080AB
- removed C10: GRM155R71A104KA01D, cvdda_5:CAPC1005X55N, symbol cboot_5:GRM155R71A104KA01D
- removed C11: GRM155R60J474KE19D, G-155_MUR, symbol cboot:GRM155R60J474KE19D
- removed C12: CL05C821JB5NNNC, CAP_CL05_SAM, symbol ccomp_5:CL05C821JB5NNNC
- removed C13: C0402C300J5GACTU, CAPC10555_55N_KEM, symbol ccomp2_5:C0402C300J5GACTU
- removed C14: GRM188R71A225KE15D, G-188_MUR, symbol cvcc_5:GRM188R71A225KE15D
- removed C15: GRM155R71A104KA01D, cvdda_5:CAPC1005X55N, symbol cvdda_5:GRM155R71A104KA01D
- removed C16, C17, C18, C19: C2012X6S1H155K125AB, CAP_2012_TDK, symbol cin_5:C2012X6S1H155K125AB
- removed C2: APXE6R3ARA101ME61G, CHEMI-E61, symbol cout:APXE6R3ARA101ME61G
- removed C20, C21, C22, C9: MSAST21GBB5106MTNA01, cout_5:CAPC2012X145N, symbol cout_5:MSAST21GBB5106MTNA01
- removed C23: 1uF, Capacitor_SMD:C_0603_1608Metric, symbol Device:C
- removed C24: 100nF, Capacitor_SMD:C_0603_1608Metric, symbol Device:C
- removed C25, C26: 10uF, Capacitor_SMD:C_0603_1608Metric, symbol Device:C
- removed C3: GRM1555C1H160JA01D, cff:CAPC1005X55N, symbol cff:GRM1555C1H160JA01D
- removed C4: GRM21BR71A225KA01L, CAP_GRM21_MUR, symbol cvcc:GRM21BR71A225KA01L
- removed C5: C1005X7R1H473K050BB, CAP_1005_TDK, symbol cinx:C1005X7R1H473K050BB
- removed C6, C8: CL32A106KBJNNNE, CAP_CL32_SAM, symbol cin:CL32A106KBJNNNE
- removed C7: UUD1V101MNL1GS, U2-P_NCH, symbol cbulk:UUD1V101MNL1GS
- removed D1: 1N5819, Diode_THT:D_DO-41_SOD81_P10.16mm_Horizontal, symbol Diode:1N5819
- removed D2: SMBJ28A, SMBJ28A:DIOM5436X244N, symbol SMBJ28A:SMBJ28A
- removed D3, D4, D5: LESD5D5.0CT1G, led:TVS_LESD5D5.0CT1G, symbol LESD5D5.0CT1G:LESD5D5.0CT1G
- removed F1: 0.1 Omh, Resistor_SMD:R_2512_6332Metric, symbol Device:Fuse
- removed IC1: IAUCN04S7L028ATMA1, IAUC120N06S5N011ATMA1, symbol M1_5:IAUCN04S7L028ATMA1
- removed J2: Conn_01x05_Socket, Connector_PinSocket_2.54mm:PinSocket_1x05_P2.54mm_Vertical, symbol Connector:Conn_01x05_Socket
- removed J3: Conn_01x15_Socket, Connector_PinSocket_2.54mm:PinSocket_1x15_P2.54mm_Vertical, symbol Connector:Conn_01x15_Socket
- removed J4: USB4105-GF-A, usb:GCT_USB4105-GF-A, symbol USB4105-GF-A:USB4105-GF-A
- removed L3: SRU8043-3R9Y, SRU80433R9Y, symbol L1:SRU8043-3R9Y
- removed R1: CRCW040243K2FKED, rfbb:RES_CRCW_0402, symbol Rfbb:CRCW040243K2FKED
- removed R10: 10k, Resistor_SMD:R_0201_0603Metric, symbol Device:R_US
- removed R11, R12: 5.1K, Resistor_SMD:R_0201_0603Metric, symbol Device:R_US
- removed R2: CRCW0402100KFKED, rcomp_5:RES_CRCW_0402, symbol rfbt:CRCW0402100KFKED
- removed R3: RC0201FR-07105KL, rpgood:RESC0603X26N, symbol rpgood:RC0201FR-07105KL
- removed R4: WSR23L000FEA, WSR, symbol rsense_5:WSR23L000FEA
- removed R5: RC0603FR-079K53L, RC0603N_YAG, symbol rt_5:RC0603FR-079K53L
- removed R6: RC0603FR-0740K2L, RC0603N_YAG, symbol rconfig_5:RC0603FR-0740K2L
- removed R8: CRCW0603100KFKEA, rpg_5:RES_CRCW_0603_VIS, symbol rpg_5:CRCW0603100KFKEA
- removed R9: CRCW060347K5FKEA, RES_CRCW_0603, symbol rvdda_5:CRCW060347K5FKEA
- removed SW1, SW2: SW_DPST_x2, Button_Switch_SMD:SW_MEC_5GSH9, symbol Switch:SW_DPST_x2
- removed U2: LM73605RNPR, LM7:QFN50P600X400X80-31N, symbol LM73605RNPR:LM73605RNPR
- removed U5: CSD17577Q5A, DQJ8, symbol M2_5:CSD17577Q5A
- removed U6: ESP32-S3-WROOM-1, RF_Module:ESP32-S3-WROOM-1, symbol RF_Module:ESP32-S3-WROOM-1
- added C1, C3, C4, C6: C2012X6S1H155K125AB, C2012X6S1H155K125AB:CAPC2012X145N, symbol cin_5:C2012X6S1H155K125AB
- added C10: CL05C821JB5NNNC, CL05C821JB5NNNC:CAPC1005X55N, symbol ccomp_5:CL05C821JB5NNNC
- added C11: C0402C300J5GACTU, CAPC10555_55N_KEM, symbol ccomp2_5:C0402C300J5GACTU
- added C12: ${SIM.PARAMS}, symbol Device:C
- added C13, C14, C15, C19, C2, C20, C33, C5, C8: C, symbol Device:C
- added C16: 10uF, symbol Device:C_Polarized
- added C17: GRM155R71A104KA01D, GRM155R71A104KA01D:CAPC1005X55N, symbol cboot_5:GRM155R71A104KA01D
- added C18, C21, C28: 100nF, symbol Device:C
- added C22: 22uF, symbol Device:C_Polarized
- added C23, C24, C25, C26: MSAST21GBB5106MTNA01, MSAST21GBB5106MTNA01:CAPC2012X145N, symbol cout_5:MSAST21GBB5106MTNA01
- added C27: 10uF, symbol Device:C
- added C29, C30: 22pF, symbol Device:C
- added C31, C32, C34: 1uF/16V, symbol Device:C
- added C7: GRM155R71A104KA01D, GRM155R71A104KA01D:CAPC1005X55N, symbol cvdda_5:GRM155R71A104KA01D
- added C9: GRM188R71A225KE15D, G-188_MUR, symbol cvcc_5:GRM188R71A225KE15D
- added D1: SMBJ28A, SMBJ28A:DIOM5436X244N, symbol SMBJ28A:SMBJ28A
- added D2: D_Schottky, symbol Device:D_Schottky
- added D3: LED, symbol Device:LED
- added F1: TR/3216TD12-R, FUS_CB_3216TD, symbol fuse:TR_3216TD12-R
- added J2: USB_C_Receptacle_USB2.0_14P, symbol Connector:USB_C_Receptacle_USB2.0_14P
- added JP1: Jumper_3_Open, symbol Jumper:Jumper_3_Open
- added L1: L, symbol Device:L
- added R1: 1M, symbol Device:R
- added R10, R11, R13, R14, R2, R21, R8: R, symbol Device:R
- added R12: RC0603FR-079K53L, RC0603N_YAG, symbol rt_5:RC0603FR-079K53L
- added R15: WSR23L000FEA, WSR, symbol rsense_5:WSR23L000FEA
- added R16, R17: 10K, symbol Device:R
- added R18: 1K, symbol Device:R
- added R19: 47.5K, symbol Device:R
- added R20: 22.1K, symbol Device:R
- added R3: CRCW060347K5FKEA, RES_CRCW_0603, symbol rvdda_5:CRCW060347K5FKEA
- added R4, R6: 5k1, symbol Device:R
- added R5: CRCW0603100KFKEA, CRCW0603100KFKEA:RESC1508X50N, symbol rpg_5:CRCW0603100KFKEA
- added R9: RC0603FR-0740K2L, RC0603N_YAG, symbol rconfig_5:RC0603FR-0740K2L
- added U1: TPD4E02B04DQA, Package_SON:USON-10_2.5x1.0mm_P0.5mm, symbol Power_Protection:TPD4E02B04DQA
- added U2: LM61460AANRJRR, LM61460AANRJRR:IC_LM61460AANRJRR, symbol lm61460AANRJRR:LM61460AANRJRR
- added U4: AMS1117-3.3, Package_TO_SOT_SMD:SOT-223-3_TabPin2, symbol Regulator_Linear:AMS1117-3.3
- added U5: ESP32-S3-WROOM-1, RF_Module:ESP32-S3-WROOM-1, symbol RF_Module:ESP32-S3-WROOM-1
- added U6: CP2102N-A02-GQFN28R, CP2102N-A02-GQFN28R:IC_CP2102N-A02-GQFN28R, symbol CP2102N-A02-GQFN28R:CP2102N-A02-GQFN28R
- J1: value 24V DC wall plug-iN -> 24; footprint Connector_BarrelJack:BarrelJack_Horizontal -> (none)
- U3: footprint LM5:QFN50P550X350X100-25N -> LM5148RGYR:QFN50P550X350X100-25N
Connections:
- net +3.3V: now also C21.1, C22.1, R14.1, U4.2 (VO)
- net +5V: now also C16.1, C18.1, U4.3 (VI)
- net GNDREF: now also C23.1, C23.2, C24.1, C24.2, C25.1, C25.2, C26.1, C26.2, R15.2
- net Heater Gnd: now also Q3.5 (Drain), Q3.6 (Drain), Q3.7 (Drain), Q3.8 (Drain); no longer Q4.5 (Drain), Q4.6 (Drain), Q4.7 (Drain), Q4.8 (Drain)
- net Heater gnd: now also Q4.5 (Drain), Q4.6 (Drain), Q4.7 (Drain), Q4.8 (Drain); no longer Q3.5 (Drain), Q3.6 (Drain), Q3.7 (Drain), Q3.8 (Drain)
- net at U3.17 (PG/SYNCOUT): now also R5.1
- net at U3.9 (VCC): now also C9.2, R5.2
- net gpio7: now reaches Q4.4 (Gate)
- net gpio6: now reaches Q5.4 (Gate)
- net at L2.2, Q1.1, Q1.2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: now also C17.1
- net at Q1.5_8, U3.12 (VIN), U3.19 (EN)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: now also C1.2, C3.2, C4.2, C6.2
- net at R7.2: now also C10.2
- net at U3.18 (PFM/SYNC), U3.8 (VDDA): now also C7.2, R3.1
- net at J1.1 (24+): now also F1.1
- net at L2.1, U3.20 (ISNS+): now also R15.1
- net at U3.4 (RT): now also R12.1
- net at U3.6 (FB): now also R3.2
- net at R7.1, U3.5 (EXTCOMP): now also C11.2
- net gpio5: now reaches Q3.4 (Gate)
- net at U3.15 (CBOOT): now also C17.2
- net at U3.3 (CNFG): now also R9.1
- net DAP renamed GND
- net GND: now also C1.1, C12.2, C16.2, C18.2, C21.2, C22.2, C27.2, C28.2, C29.2, C3.1, C30.2, C31.2, C32.2, C33.2, C34.2, C4.1, C6.1, C7.1, C9.1, D1.A, D1.C, D3.1 (K), F1.2, J2.A1 (GND), J2.A12 (GND), J2.B1 (GND), J2.B12 (GND), R1.2, R12.2, R19.2, R21.2, R4.2, R6.2, R9.2, U1.3 (G), U1.8 (G), U4.1 (GND), U5.1 (GND), U5.40 (GND), U5.41 (GND), U6.29 (EXP), U6.3 (GND)
- new net: C13.2, C15.2, C2.2, C20.2, C5.2, C8.2, R11.2, R2.1, U2.11 (PGND2), U2.3 (AGND), U2.9 (PGND1)
- new net: J2.B5 (CC2), R4.1
- new net: C14.1, U2.13 (RBOOT), U2.14 (CBOOT)
- new net: C14.2, L1.1, U2.10 (SW)
- new net: C5.1, U2.2 (VCC)
- new net: R21.1, U6.11 (~{SUSPEND})
- new net: R10.2, R11.1, R13.1, U2.4 (FB)
- new net: C19.2, R13.2
- new net: C10.1, C11.1
- new net: R8.1, U2.5 (PGOOD)
- new net: R2.2, U2.6 (RT)
- new net: C27.1, C28.1, U5.2 (3V3)
- new net: D2.2 (A), J2.A4 (VBUS), J2.A9 (VBUS), J2.B4 (VBUS), J2.B9 (VBUS)
- new net: D3.2 (A), R14.2
- new net: C33.1, U6.6 (VDD), U6.7 (VREGIN)
- new net: C34.1, R19.1, R20.2, U6.8 (VBUS)
- new net: J2.S1 (SHIELD), R1.1
- new net: J2.A5 (CC1), R6.1
- new net: R18.1, U6.9 (~{RST})
- new net +5V_usb: D2.1 (K), JP1.3 (B), U1.1 (IO1)
- new net 3.3V_bat: JP1.1 (A)
- new net 5V_bat: C19.1, C20.1, L1.2, R10.1, R8.2, U2.1 (BIAS)
- new net BOOT: C32.1, R17.2, U5.27 (IO0)
- new net Battery: C13.1, C15.1, C2.1, C8.1, U2.12 (VIN2), U2.8 (VIN1)
- new net CHB_2: U5.23 (IO21)
- new net CHIP_PU: C31.1, R16.2, U5.3 (EN)
- new net Data+: C29.1, J2.A6 (D+), J2.B6 (D+), U1.4 (IO3), U5.14 (USB_D+)
- new net Data-: C30.1, J2.A7 (D-), J2.B7 (D-), U1.5 (IO4), U5.13 (USB_D-)
- new net SCL: U5.38 (IO2)
- new net SDA: U5.39 (IO1)
- new net dtr: U6.28 (DTR)
- new net rts: U6.24 (RTS)
- new net uorxd: U6.25 (RXD)
- new net uotxd: U6.26 (TXD)
- no-connect marks 12 -> 15
Other:
- note removed: "3.3V Buck"
- note removed: "SCREW TERMINALS"

Commit message: libary update 75% footprints added
Parts:
- removed C1, C3, C4, C6: C2012X6S1H155K125AB, C2012X6S1H155K125AB:CAPC2012X145N, symbol cin_5:C2012X6S1H155K125AB
- removed C12: ${SIM.PARAMS}, symbol Device:C
- removed C13, C15: C, symbol Device:C
- removed C24, C25, C26: MSAST21GBB5106MTNA01, MSAST21GBB5106MTNA01:CAPC2012X145N, symbol cout_5:MSAST21GBB5106MTNA01
- removed C32: 1uF/16V, symbol Device:C
- removed C7: GRM155R71A104KA01D, GRM155R71A104KA01D:CAPC1005X55N, symbol cvdda_5:GRM155R71A104KA01D
- removed D1: SMBJ28A, SMBJ28A:DIOM5436X244N, symbol SMBJ28A:SMBJ28A
- removed F1: TR/3216TD12-R, FUS_CB_3216TD, symbol fuse:TR_3216TD12-R
- removed J1: 24, symbol Connector_Generic:Conn_01x02
- removed Q1: CSD18512Q5B, CSD18512Q5B:TRANS_CSD18512Q5B, symbol CSD18512Q5B:CSD18512Q5B
- removed Q3, Q4, Q5: RQ3E110AJTB, HSMT8_ROM, symbol rq3e11oajtbct:RQ3E110AJTB
- removed R17: 10K, symbol Device:R
- removed R3: CRCW060347K5FKEA, RES_CRCW_0603, symbol rvdda_5:CRCW060347K5FKEA
- removed Vin1: dc, symbol Device:Battery
- added C1, C3, C4, C6: C2012X6S1H155K125AB, footprints:CAP_2012_TDK-L, symbol BreadBoard:C2012X6S1H155K125AB
- added C12, C24, C25: MSAST21GBB5106MTNA01, footprints:CAPC2012X145N, symbol BreadBoard:MSAST21GBB5106MTNA01
- added C13, C35: GRM32ER71H475KA88L, footprints:CAPC3225X270N, symbol BreadBoard:GRM32ER71H475KA88L
- added C26, C34: C, symbol Device:C
- added C7: GRM155R71A104KA01D, footprints:G-155_MUR-L, symbol BreadBoard:GRM155R71A104KA01D
- added D1: SMBJ28A, footprints:DIOM5436X244N, symbol BreadBoard:SMBJ28A
- added F1: TR/3216TD12-R, footprints:FUS_CB_3216TD, symbol BreadBoard:TR_3216TD12-R
- added J1: PD-40, footprints:CUI_PD-40, symbol BreadBoard:PD-40
- added J3: Conn_01x02_Pin, symbol Connector:Conn_01x02_Pin
- added Q1, Q2: BC818, Package_TO_SOT_SMD:SOT-23, symbol Transistor_BJT:BC818
- added Q3: CSD18512Q5B, footprints:TRANS_CSD18512Q5B, symbol BreadBoard:CSD18512Q5B
- added Q5, Q6: RQ3E110AJTB, footprints:HSMT8_ROM-L, symbol BreadBoard:RQ3E110AJTB
- added R10, R12, R13, R9: R, symbol Device:R
- added R25, R26: 47, symbol Device:R
- added R27, R28: 100k, symbol Device:R
- added R29: 0, symbol Device:R
- added R3: CRCW060347K5FKEA, footprints:RES_CRCW_0603-L, symbol BreadBoard:CRCW060347K5FKEA
- added SW1, SW2: SKRPADE010, footprints:SKRPADE010_AAL, symbol BreadBoard:SKRPADE010
- C10: footprint CL05C821JB5NNNC:CAPC1005X55N -> footprints:CAP_CL05_SAM-L; symbol ccomp_5:CL05C821JB5NNNC -> BreadBoard:CL05C821JB5NNNC
- C11: footprint CAPC10555_55N_KEM -> footprints:CAPC10555_55N_KEM-L; symbol ccomp2_5:C0402C300J5GACTU -> BreadBoard:C0402C300J5GACTU
- C14: value C -> GRM155R71A104KA01D; footprint (none) -> footprints:CAPC1005X55N
- C17: footprint GRM155R71A104KA01D:CAPC1005X55N -> footprints:G-155_MUR-L; symbol cboot_5:GRM155R71A104KA01D -> BreadBoard:GRM155R71A104KA01D
- C2: value C -> GRM188R60J105KA01D; footprint (none) -> footprints:G-188_MUR-L
- C23: footprint MSAST21GBB5106MTNA01:CAPC2012X145N -> footprints:CAPC2012X145N; symbol cout_5:MSAST21GBB5106MTNA01 -> BreadBoard:MSAST21GBB5106MTNA01
- C33: footprint (none) -> Capacitor_SMD:C_0201_0603Metric_Pad0.64x0.40mm_HandSolder
- C5, C8: value C -> C1005X5R1V474K050BC; footprint (none) -> footprints:CAPC1005X55N
- C9: footprint G-188_MUR -> footprints:G-188_MUR-L; symbol cvcc_5:GRM188R71A225KE15D -> BreadBoard:GRM188R71A225KE15D
- D2: footprint (none) -> Diode_SMD:D_SOD-523
- J2: footprint (none) -> Connector_USB:USB_C_Receptacle_HRO_TYPE-C-31-M-12
- JP1: footprint (none) -> Connector_Samtec_HPM_THT:Samtec_HPM-03-01-x-S_Straight_1x03_Pitch5.08mm
- L1: footprint (none) -> footprints:WE-XHMI_5050
- L2: footprint IND_CDEP63MENP-R68MC_SUM -> footprints:IND_CDEP63MENP-R68MC_SUM-L; symbol L1_5:CDEP63MENP-R68MC -> BreadBoard:CDEP63MENP-R68MC
- Q4: renamed from Q2; footprint CSD18512Q5B:TRANS_CSD18512Q5B -> footprints:TRANS_CSD18512Q5B; symbol CSD18512Q5B:CSD18512Q5B -> BreadBoard:CSD18512Q5B
- R1, R4, R6: footprint (none) -> Resistor_SMD:R_0201_0603Metric_Pad0.64x0.40mm_HandSolder
- R11: renamed from R9; footprint RC0603N_YAG -> footprints:RC0603N_YAG-L; symbol rconfig_5:RC0603FR-0740K2L -> BreadBoard:RC0603FR-0740K2L
- R14: renamed from R10; footprint (none) -> footprints:RES_CRCW_0402_VIS-L
- R16: renamed from R12; footprint RC0603N_YAG -> footprints:RC0603N_YAG-L; symbol rt_5:RC0603FR-079K53L -> BreadBoard:RC0603FR-079K53L
- R18: renamed from R14; value R -> 10k; footprint (none) -> Resistor_SMD:R_0603_1608Metric_Pad0.98x0.95mm_HandSolder
- R19: renamed from R15; footprint WSR -> footprints:WSR-L; symbol rsense_5:WSR23L000FEA -> BreadBoard:WSR23L000FEA
- R2: footprint (none) -> footprints:RESC2012X50N
- R24: renamed from R21; value R -> 10k
- R5: footprint CRCW0603100KFKEA:RESC1508X50N -> footprints:RES_CRCW_0603_VIS-L; symbol rpg_5:CRCW0603100KFKEA -> BreadBoard:CRCW0603100KFKEA
- R7: footprint RES_CRCW_0402 -> footprints:RES_CRCW_0402-L; symbol rcomp_5:CRCW04024K87FKED -> BreadBoard:CRCW04024K87FKED
- R8: footprint (none) -> footprints:RES_CRCW_0402_VIS-L
- U2: footprint LM61460AANRJRR:IC_LM61460AANRJRR -> footprints:IC_LM61460AANRJRR; symbol lm61460AANRJRR:LM61460AANRJRR -> BreadBoard:LM61460AANRJRR
- U3: footprint LM5148RGYR:QFN50P550X350X100-25N -> footprints:QFN50P550X350X100-25N; symbol LM5148RGYR:LM5148RGYR -> BreadBoard:LM5148RGYR
- U6: footprint CP2102N-A02-GQFN28R:IC_CP2102N-A02-GQFN28R -> footprints:IC_CP2102N-A02-GQFN28R; symbol CP2102N-A02-GQFN28R:CP2102N-A02-GQFN28R -> BreadBoard:CP2102N-A02-GQFN28R
- renumbered C34 to C31, C31 to C32, R11 to R15, R13 to R17, R19 to R21, R18 to R22, R16 to R23
Connections:
- net +5V is gone; now on net +5V_Jump: C16.1, C18.1, U4.3 (VI)
- net 5V_bat is gone; now on net +5V_input: C19.1, C20.1, L1.2, R14.1, R8.2, U2.1 (BIAS)
- net uorxd is gone; now on net U0RXD: U6.25 (RXD)
- net uotxd is gone; now on net U0TXD: U6.26 (TXD)
- net +3.3V: now also C27.1, C28.1, C33.1, R22.2, U6.6 (VDD), U6.7 (VREGIN), R29.1
- net BOOT: now also C26.1, R13.2, SW2.1
- net CHIP_PU: now also C34.1, R12.2, SW1.1
- net Data+: no longer U5.14 (USB_D+)
- net Data-: no longer U5.13 (USB_D-)
- net GND: now also C2.2, C20.2, C23.1, C5.2, C8.2, R15.2, R2.1, U2.11 (PGND2), U2.3 (AGND), U2.9 (PGND1), C1.1, C12.1, C13.1, C24.1, C25.1, C26.2, C3.1, C34.2, C35.1, C4.1, C6.1, C7.1, D1.A, J1.3, J1.4, J1.S1 (SHIELD), Q5.1, Q5.2, Q5.3, Q6.1, Q6.2, Q6.3, R27.1, R28.1, SW1.3, SW2.3
- net SCL: now also J3.2 (Pin_2)
- net SDA: now also J3.1 (Pin_1)
- net dtr: now also Q2.3 (C), R9.1
- net gpio6: now also U5.6 (IO6), R25.1
- net gpio7: now also U5.7 (IO7), R26.1
- net rts: now also Q1.2 (E), R10.2
- net at C17.1, L2.2, Q4.5_8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: now also Q3.1, Q3.2, Q3.3
- net at U2.2 (VCC): now also C2.1; no longer C5.1
- net at C9.2, U3.9 (VCC): now also R5.1; no longer R5.2
- net at U3.18 (PFM/SYNC), U3.8 (VDDA): now also C7.2, R3.1
- net +VBUS: now reaches U3.12 (VIN), U3.19 (EN)
- net +VBUS: now also C5.1, C8.1, U2.12 (VIN2), U2.8 (VIN1), C1.2, C13.2, C3.2, C35.2, C4.2, C6.2, D1.C, F1.2, Q3.5_8
- net +5V_Jump: now reaches JP1.2 (C)
- net +5V_Jump: now also R20.1
- net at U3.17 (PG/SYNCOUT): now also R5.2; no longer R5.1
- net at U3.13 (HO): now also Q3.4
- net at U3.6 (FB): now also R3.2
- net U0RXD: now reaches U5.36 (RXD0)
- net U0TXD: now reaches U5.37 (TXD0)
- net +3.3V_esp: now reaches R23.1
- net +3.3V_esp: now also U5.2 (3V3), R29.2
- net 3.3V_bat renamed +5V_input
- removed net Battery: C2.1, C8.1, U2.12 (VIN2), U2.8 (VIN1)
- net CHB_2: no longer names the net of U5.23 (IO21)
- net GNDREF renamed Heater Vcc 1
- net Heater Vcc 1: now also C12.2, C24.2, C25.2; no longer C23.1
- new net: Q5.4, R26.2, R28.2
- new net: Q2.1 (B), R10.1
- new net: Q6.4, R25.2, R27.2
- new net: Q1.1 (B), R9.2
- new net: Q1.3 (C), R12.1
- new net: Q2.2 (E), R13.1
- new net: F1.1, J1.1, J1.2
- new net Heater_1: Q5.5, Q5.6, Q5.7, Q5.8
- new net Heater_2: Q6.5, Q6.6, Q6.7, Q6.8
- no-connect marks 15 -> 52
Other:
- moved on the sheet: C10, C31, C33, C8, R2, R20, R21, R22, R24, R7, U6

Commit message: updates
Parts:
- C16: value 10uF -> GRM155R61A106ME11D; footprint (none) -> footprints:RC0603N_YAG-L
- C18, C21: value 100nF -> C0201X5R104K100NTA; footprint (none) -> footprints:RC0603N_YAG-L
- C19: value C -> CC0805JRNPO9BN120; footprint (none) -> footprints:CAP_CC0805_YAG-L
- C20: value C -> GRM31CR61A107MEA8K; footprint (none) -> footprints:CAPC3216X190N
- C22: value 22uF -> GRM188R61A226ME15D; footprint (none) -> footprints:RC0603N_YAG-L
- L1: value L -> WE-XHMI_5050
- R14, R8: value R -> CRCW0402100KFKED
- R15: value R -> RC0603FR-0724K9L; footprint (none) -> footprints:RC0603N_YAG-L
- R17: value R -> CRCW04021K00FKED; footprint (none) -> footprints:RESC1005X40N
- R18: value 10k -> 150
- R2: value R -> GRM188R60J105KA01D
Changed lines of the file:
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@@
 		(on_board yes)
 		(dnp no)
-		(fields_autoplaced yes)
 		(property "Reference" "R17"
-			(at 237.49 224.79 90)
+			(at 237.49 227.584 90)
 			(effects
 				(font
@@
 			)
 		)
-		(property "Value" "R"
+		(property "Value" "CRCW04021K00FKED"
 			(at 237.49 227.33 90)
 			(effects
@@
 					(size 1.27 1.27)
 				)
+				(hide yes)
 			)
 		)
-		(property "Footprint" ""
+		(property "Footprint" "footprints:RESC1005X40N"
 			(at 237.49 232.918 90)
 			(effects
@@
 			)
 		)
-		(property "Value" "C"
+		(property "Value" "CC0805JRNPO9BN120"
 			(at 250.19 219.7099 0)
 			(effects
@@
 				)
 				(justify left)
+				(hide yes)
 			)
 		)
-		(property "Footprint" ""
+		(property "Footprint" "footprints:CAP_CC0805_YAG-L"
 			(at 247.3452 222.25 0)
 			(effects
@@
 				)
 				(justify left)
+				(hide yes)
 			)
 		)
@@
 			)
 		)
-		(property "Value" "10k"
+		(property "Value" "150"
 			(at 303.53 91.4399 0)
 			(effects
@@
 			)
 		)
-		(property "Value" "L"
+		(property "Value" "WE-XHMI_5050"
 			(at 205.74 208.28 90)
 			(effects
@@
 					(size 1.27 1.27)
 				)
+				(hide yes)
 			)
 		)
@@
 		(on_board yes)
 		(dnp no)
-		(fields_autoplaced yes)
 		(property "Reference" "C21"
 			(at 275.59 88.8999 0)
@@
 			)
 		)
-		(property "Value" "100nF"
-			(at 275.59 91.4399 0)
+		(property "Value" "C0201X5R104K100NTA"
+			(at 263.398 105.156 0)
 			(effects
 				(font
@@
 			)
 		)
-		(property "Footprint" ""
+		(property "Footprint" "footprints:RC0603N_YAG-L"
 			(at 272.7452 93.98 0)
 			(effects
@@
 			)
 		)
-		(property "Value" "R"
+		(property "Value" "GRM188R60J105KA01D"
 			(at 93.98 237.4899 0)
 			(effects
@@
 				)
 				(justify right)
+				(hide yes)
 			)
 		)
@@
 			)
 		)
-		(property "Value" "R"
+		(property "Value" "CRCW0402100KFKED"
 			(at 228.6 222.2499 0)
 			(effects
@@
 				)
 				(justify left)
+				(hide yes)
 			)
 		)
@@
 				)
 				(justify left)
+				(hide yes)
 			)
 		)
@@
 				)
 				(justify left)
+				(hide yes)
 			)
 		)
@@
 			)
 		)
-		(property "Value" "C"
+		(property "Value" "GRM31CR61A107MEA8K"
 			(at 265.43 231.1399 0)
 			(effects
@@
 				)
 				(justify left)
+				(hide yes)
 			)
 		)
-		(property "Footprint" ""
+		(property "Footprint" "footprints:CAPC3216X190N"
 			(at 262.5852 233.68 0)
 			(effects
@@
 				)
 				(justify left)
+				(hide yes)
 			)
 		)
@@
 		(on_board yes)
 		(dnp no)
-		(fields_autoplaced yes)
 		(property "Reference" "C22"
 			(at 289.56 88.0109 0)
@@
 			)
 		)
-		(property "Value" "22uF"
-			(at 289.56 90.5509 0)
+		(property "Value" "GRM188R61A226ME15D"
+			(at 273.558 110.236 0)
 			(effects
 				(font
@@
 			)
 		)
-		(property "Footprint" ""
+		(property "Footprint" "footprints:RC0603N_YAG-L"
 			(at 286.7152 93.98 0)
 			(effects
@@
 		(on_board yes)
 		(dnp no)
-		(fields_autoplaced yes)
 		(property "Reference" "C18"
 			(at 240.03 88.8999 0)
@@
 			)
 		)
-		(property "Value" "100nF"
-			(at 240.03 91.4399 0)
+		(property "Value" "C0201X5R104K100NTA"
+			(at 222.504 82.042 0)
 			(effects
 				(font
@@
 			)
 		)
-		(property "Footprint" ""
+		(property "Footprint" "footprints:RC0603N_YAG-L"
 			(at 237.1852 93.98 0)
 			(effects
@@
 				)
 				(justify left)
+				(hide yes)
 			)
 		)
@@
 			)
 		)
-		(property "Value" "R"
+		(property "Value" "CRCW0402100KFKED"
 			(at 134.62 237.49 90)
 			(effects
@@
 					(size 1.27 1.27)
 				)
+				(hide yes)
 			)
 		)
@@
 		(on_board yes)
 		(dnp no)
-		(fields_autoplaced yes)
 		(property "Reference" "C16"
 			(at 224.79 89.2809 0)
@@
 			)
 		)
-		(property "Value" "10uF"
-			(at 224.79 91.8209 0)
+		(property "Value" "GRM155R61A106ME11D"
+			(at 194.818 93.472 0)
 			(effects
 				(font
@@
 			)
 		)
-		(property "Footprint" ""
+		(property "Footprint" "footprints:RC0603N_YAG-L"
 			(at 221.9452 95.25 0)
 			(effects
@@
 			)
 		)
-		(property "Value" "R"
+		(property "Value" "RC0603FR-0724K9L"
 			(at 228.6 241.2999 0)
 			(effects
@@
 				)
 				(justify left)
+				(hide yes)
 			)
 		)
-		(property "Footprint" ""
+		(property "Footprint" "footprints:RC0603N_YAG-L"
 			(at 224.282 240.03 90)
 			(effects

Commit message: layout!
Parts:
- removed C29, C30: 22pF, symbol Device:C
- removed C31: 1uF/16V, symbol Device:C
- removed C33: C, Capacitor_SMD:C_0201_0603Metric_Pad0.64x0.40mm_HandSolder, symbol Device:C
- removed Q1, Q2: BC818, Package_TO_SOT_SMD:SOT-23, symbol Transistor_BJT:BC818
- removed R10, R12, R13: R, symbol Device:R
- removed R20: 22.1K, symbol Device:R
- removed R21: 47.5K, symbol Device:R
- removed R22: 1K, symbol Device:R
- removed R24: 10k, symbol Device:R
- removed R29: 0, symbol Device:R
- removed U6: CP2102N-A02-GQFN28R, footprints:IC_CP2102N-A02-GQFN28R, symbol BreadBoard:CP2102N-A02-GQFN28R
- added C15: GRM033R61A104KE15D, footprints:CAPC0603X33N, symbol Device:C
- C16: value GRM155R61A106ME11D -> 10uF
- C18, C21: value C0201X5R104K100NTA -> 100nF
- C22: value GRM188R61A226ME15D -> 22uF
- C26, C34: value C -> 0402B104K500HI; footprint (none) -> Capacitor_SMD:C_0402_1005Metric_Pad0.74x0.62mm_HandSolder
- C27: footprint (none) -> footprints:G-155_MUR-L
- C28, C32: footprint (none) -> footprints:CAPC0603X33N
- D3: footprint (none) -> LED_SMD:LED_0201_0603Metric
- J3: footprint (none) -> Connector_PinHeader_1.00mm:PinHeader_1x02_P1.00mm_Vertical
- R1: value 1M -> 10k; footprint Resistor_SMD:R_0201_0603Metric_Pad0.64x0.40mm_HandSolder -> Resistor_SMD:R_0201_0603Metric
- R23: footprint (none) -> Resistor_SMD:R_0201_0603Metric
- R25, R26, R27, R28: footprint (none) -> Resistor_SMD:R_0201_0603Metric_Pad0.64x0.40mm_HandSolder
- R9: value R -> 10k; footprint (none) -> Resistor_SMD:R_0201_0603Metric
Connections:
- net +3.3V_esp is gone; now on net +3.3V: R23.1, U5.2 (3V3)
- net dtr is gone; now on net +3.3V: R9.1
- net +3.3V: now also R1.1
- net +5V_usb: now also C15.1
- net BOOT: now also R9.2
- net CHIP_PU: now also R1.2
- net Data+: now also U5.14 (USB_D+)
- net Data-: now also U5.13 (USB_D-)
- net GND: now also J1.2, J2.S1 (SHIELD), C15.2; no longer J1.4, R1.2
- net at F1.1, J1.1: now also J1.4; no longer J1.2
- net U0RXD: no longer names the net of U5.36 (RXD0)
- net U0TXD: no longer names the net of U5.37 (TXD0)
- no-connect marks 52 -> 35
Other:
- moved on the sheet: C1, C10, C11, C12, C13, C14, C16, C17, C18, C19, C2, C20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
