File: BreadBoard_git/BreadBoard_git.kicad_sch (KiCad schematic)
At the start: 73 parts, among them J1 PD-40, J2 USB_C_Receptacle_USB2.0_14P, J3 Conn_01x02_Pin, Q3 CSD18512Q5B, Q4 CSD18512Q5B, Q5 RQ3E110AJTB, Q6 RQ3E110AJTB, SW1 SKRPADE010, SW2 SKRPADE010, U1 TPD4E02B04DQA, U2 LM61460AANRJRR, U3 LM5148RGYR, U4 AMS1117-3.3, U5 ESP32-S3-WROOM-1

Commit message: update!
Parts:
- removed C1, C3, C4, C6: C2012X6S1H155K125AB, footprints:CAP_2012_TDK-L, symbol BreadBoard:C2012X6S1H155K125AB
- removed C10: CL05C821JB5NNNC, footprints:CAP_CL05_SAM-L, symbol BreadBoard:CL05C821JB5NNNC
- removed C11: C0402C300J5GACTU, footprints:CAPC10555_55N_KEM-L, symbol BreadBoard:C0402C300J5GACTU
- removed C12, C23, C24, C25: MSAST21GBB5106MTNA01, footprints:CAPC2012X145N, symbol BreadBoard:MSAST21GBB5106MTNA01
- removed C13, C35: GRM32ER71H475KA88L, footprints:CAPC3225X270N, symbol BreadBoard:GRM32ER71H475KA88L
- removed C14: GRM155R71A104KA01D, footprints:CAPC1005X55N, symbol Device:C
- removed C15: GRM033R61A104KE15D, footprints:CAPC0603X33N, symbol Device:C
- removed C16: 10uF, footprints:RC0603N_YAG-L, symbol Device:C_Polarized
- removed C17, C7: GRM155R71A104KA01D, footprints:G-155_MUR-L, symbol BreadBoard:GRM155R71A104KA01D
- removed C18, C21: 100nF, footprints:RC0603N_YAG-L, symbol Device:C
- removed C19: CC0805JRNPO9BN120, footprints:CAP_CC0805_YAG-L, symbol Device:C
- removed C20: GRM31CR61A107MEA8K, footprints:CAPC3216X190N, symbol Device:C
- removed C22: 22uF, footprints:RC0603N_YAG-L, symbol Device:C_Polarized
- removed C26, C34: 0402B104K500HI, Capacitor_SMD:C_0402_1005Metric_Pad0.74x0.62mm_HandSolder, symbol Device:C
- removed C9: GRM188R71A225KE15D, footprints:G-188_MUR-L, symbol BreadBoard:GRM188R71A225KE15D
- removed J3: Conn_01x02_Pin, Connector_PinHeader_1.00mm:PinHeader_1x02_P1.00mm_Vertical, symbol Connector:Conn_01x02_Pin
- removed JP1: Jumper_3_Open, Connector_Samtec_HPM_THT:Samtec_HPM-03-01-x-S_Straight_1x03_Pitch5.08mm, symbol Jumper:Jumper_3_Open
- removed L1: WE-XHMI_5050, footprints:WE-XHMI_5050, symbol Device:L
- removed L2: CDEP63MENP-R68MC, footprints:IND_CDEP63MENP-R68MC_SUM-L, symbol BreadBoard:CDEP63MENP-R68MC
- removed Q3, Q4: CSD18512Q5B, footprints:TRANS_CSD18512Q5B, symbol BreadBoard:CSD18512Q5B
- removed R11: RC0603FR-0740K2L, footprints:RC0603N_YAG-L, symbol BreadBoard:RC0603FR-0740K2L
- removed R14, R8: CRCW0402100KFKED, footprints:RES_CRCW_0402_VIS-L, symbol Device:R
- removed R15: RC0603FR-0724K9L, footprints:RC0603N_YAG-L, symbol Device:R
- removed R16: RC0603FR-079K53L, footprints:RC0603N_YAG-L, symbol BreadBoard:RC0603FR-079K53L
- removed R17: CRCW04021K00FKED, footprints:RESC1005X40N, symbol Device:R
- removed R19: WSR23L000FEA, footprints:WSR-L, symbol BreadBoard:WSR23L000FEA
- removed R3: CRCW060347K5FKEA, footprints:RES_CRCW_0603-L, symbol BreadBoard:CRCW060347K5FKEA
- removed R5: CRCW0603100KFKEA, footprints:RES_CRCW_0603_VIS-L, symbol BreadBoard:CRCW0603100KFKEA
- removed R7: CRCW04024K87FKED, footprints:RES_CRCW_0402-L, symbol BreadBoard:CRCW04024K87FKED
- removed R9: 10k, Resistor_SMD:R_0201_0603Metric, symbol Device:R
- added C1: 10uF, Capacitor_SMD:C_0603_1608Metric_Pad1.08x0.95mm_HandSolder, symbol Device:C
- added C3, C4, C6: 0u1F, Capacitor_SMD:C_0603_1608Metric_Pad1.08x0.95mm_HandSolder, symbol Device:C
- added C7: 22pF, Capacitor_SMD:C_0402_1005Metric_Pad0.74x0.62mm_HandSolder, symbol Device:C
- added Cboot1: 0.1 µF, Resistor_SMD:R_0402_1005Metric_Pad0.72x0.64mm_HandSolder, symbol Device:C
- added Cboot2: .1uF, Capacitor_SMD:C_0201_0603Metric_Pad0.64x0.40mm_HandSolder, symbol Device:C
- added Ccomp1: 3.3nF, Capacitor_SMD:C_0402_1005Metric_Pad0.74x0.62mm_HandSolder, symbol Device:C
- added Cff1: 33pF, Capacitor_SMD:C_0201_0603Metric_Pad0.64x0.40mm_HandSolder, symbol Device:C
- added Chf1: 33pF, Capacitor_SMD:C_0402_1005Metric_Pad0.74x0.62mm_HandSolder, symbol Device:C
- added Cin-hf1, Cin-hf2: 220nF, Capacitor_SMD:C_0603_1608Metric_Pad1.08x0.95mm_HandSolder, symbol Device:C
- added Cin1, Cin2, Cin3, Cin4, Cinblk1: 10uF, Capacitor_SMD:C_1210_3225Metric_Pad1.33x2.70mm_HandSolder, symbol Device:C
- added Cin5, Cin6, Cin7, Cin8, Cout9: .1uF, Capacitor_SMD:C_0402_1005Metric_Pad0.74x0.62mm_HandSolder, symbol Device:C
- added Cout1, Cout2, Cout3, Cout4: 22uF, Capacitor_SMD:C_1210_3225Metric_Pad1.33x2.70mm_HandSolder, symbol Device:C
- added Cout5: 47uf, Capacitor_SMD:C_1210_3225Metric_Pad1.33x2.70mm_HandSolder, symbol Device:C
- added Cout6: 47uF, Capacitor_SMD:C_1210_3225Metric_Pad1.33x2.70mm_HandSolder, symbol Device:C
- added Cvcc1: 2.2uF, Capacitor_SMD:C_0603_1608Metric_Pad1.08x0.95mm_HandSolder, symbol Device:C
- added Cvcc2: 1uF, Capacitor_SMD:C_0603_1608Metric_Pad1.08x0.95mm_HandSolder, symbol Device:C
- added Cvdda1: 0.47uF, Capacitor_SMD:C_0402_1005Metric_Pad0.74x0.62mm_HandSolder, symbol Device:C
- added Cvin1: 22nF, Capacitor_SMD:C_0603_1608Metric_Pad1.08x0.95mm_HandSolder, symbol Device:C
- added J4, J5: Conn_01x02_Pin, Connector_PinHeader_2.54mm:PinHeader_1x02_P2.54mm_Vertical, symbol Connector:Conn_01x02_Pin
- added J7: Conn_01x15_Pin, Connector_PinHeader_2.54mm:PinHeader_1x15_P2.54mm_Vertical, symbol Connector:Conn_01x15_Pin
- added J8: Conn_01x05_Pin, Connector_PinHeader_2.54mm:PinHeader_1x05_P2.54mm_Vertical, symbol Connector:Conn_01x05_Pin
- added JP1: Jumper_3_Bridged12, Connector_PinHeader_2.54mm:PinHeader_1x03_P2.54mm_Vertical, symbol Jumper:Jumper_3_Bridged12
- added Lout1: 4.7u, footprints:WSR-L, symbol Device:L
- added Lout2: 22uF, footprints:IND_NS12565T100MNV_TAY, symbol Device:L
- added Q1, Q2: NMOS, footprints:TRANS_CSD18512Q5B, symbol Simulation_SPICE:NMOS
- added R3: 100k, Resistor_SMD:R_0402_1005Metric_Pad0.72x0.64mm_HandSolder, symbol Device:R
- added Rcnfg1: 29.4k, Resistor_SMD:R_0402_1005Metric_Pad0.72x0.64mm_HandSolder, symbol Device:R
- added Rcomp1: 11.8k, Resistor_SMD:R_0402_1005Metric_Pad0.72x0.64mm_HandSolder, symbol Device:R
- added Rent1: 255k, Resistor_SMD:R_0603_1608Metric_Pad0.98x0.95mm_HandSolder, symbol Device:R
- added Rfb1: 48.7k, Resistor_SMD:R_0402_1005Metric_Pad0.72x0.64mm_HandSolder, symbol Device:R
- added Rfbb1: 24.9k, Resistor_SMD:R_0603_1608Metric_Pad0.98x0.95mm_HandSolder, symbol Device:R
- added Rfbt1, Rpg1, Rrenb1: 100k, Resistor_SMD:R_0603_1608Metric_Pad0.98x0.95mm_HandSolder, symbol Device:R
- added Rff1: 1k, Resistor_SMD:R_0603_1608Metric_Pad0.98x0.95mm_HandSolder, symbol Device:R
- added Rrt1: 54.9k, Resistor_SMD:R_0402_1005Metric_Pad0.72x0.64mm_HandSolder, symbol Device:R
- added Rrt2: 33.2k, Resistor_SMD:R_0603_1608Metric_Pad0.98x0.95mm_HandSolder, symbol Device:R
- added Rs1: 4.3m, Resistor_SMD:R_0508_1220Metric_Pad1.12x2.15mm_HandSolder, symbol Device:R
- added Ruv1: 200k, Resistor_SMD:R_0402_1005Metric_Pad0.72x0.64mm_HandSolder, symbol Device:R
- added Ruv2: 9.53k, Resistor_SMD:R_0402_1005Metric_Pad0.72x0.64mm_HandSolder, symbol Device:R
- added TP1: 24V_in, TestPoint:TestPoint_Keystone_5019_Miniature, symbol Connector:TestPoint
- added TP2: TestPoint:TestPoint_Keystone_5019_Miniature, symbol Connector:TestPoint
- added TP3: 12V_out, TestPoint:TestPoint_Keystone_5019_Miniature, symbol Connector:TestPoint
- added TP4: 12V_out_gnd, TestPoint:TestPoint_Keystone_5019_Miniature, symbol Connector:TestPoint
- C2: value GRM188R60J105KA01D -> 10uF; footprint footprints:G-188_MUR-L -> Capacitor_SMD:C_0603_1608Metric_Pad1.08x0.95mm_HandSolder
- C27: footprint footprints:G-155_MUR-L -> Capacitor_SMD:C_0805_2012Metric_Pad1.18x1.45mm_HandSolder
- C28: value 100nF -> 0u1F; footprint footprints:CAPC0603X33N -> Capacitor_SMD:C_0603_1608Metric_Pad1.08x0.95mm_HandSolder
- C32: footprint footprints:CAPC0603X33N -> Capacitor_SMD:C_0603_1608Metric_Pad1.08x0.95mm_HandSolder
- C5: value C1005X5R1V474K050BC -> 0u1F; footprint footprints:CAPC1005X55N -> Capacitor_SMD:C_0603_1608Metric_Pad1.08x0.95mm_HandSolder
- C8: value C1005X5R1V474K050BC -> 22pF; footprint footprints:CAPC1005X55N -> Capacitor_SMD:C_0402_1005Metric_Pad0.74x0.62mm_HandSolder
- D2: footprint Diode_SMD:D_SOD-523 -> Diode_SMD:D_0603_1608Metric_Pad1.05x0.95mm_HandSolder
- F1: value TR/3216TD12-R -> 0680L6300-05; footprint footprints:FUS_CB_3216TD -> footprints:FUSC6125X279N
- R1, R23: footprint Resistor_SMD:R_0201_0603Metric -> Resistor_SMD:R_0603_1608Metric_Pad0.98x0.95mm_HandSolder
- R18: value 150 -> 75
- R2: value GRM188R60J105KA01D -> 10k; footprint footprints:RESC2012X50N -> Resistor_SMD:R_0603_1608Metric_Pad0.98x0.95mm_HandSolder
- R25, R26, R27, R28: footprint Resistor_SMD:R_0201_0603Metric_Pad0.64x0.40mm_HandSolder -> Resistor_SMD:R_0603_1608Metric_Pad0.98x0.95mm_HandSolder
Connections:
- net +3.3V: now also C2.2, R2.1, C3.1, J7.1 (Pin_1), J8.1 (Pin_1)
- net BOOT: now also R2.2, C6.1
- net CHIP_PU: now also C5.1
- net GND: now also C2.1, U3.18 (PFM/SYNC), C1.2, C3.2, C4.2, C6.2, C7.2, Cin-hf1.2, Cin-hf2.2, Cin1.2, Cin2.2, Cin3.2, Cin4.2, Cin5.2, Cin6.2, Cin7.2, Cin8.2, Cinblk1.2, Cout1.2, Cout2.2, Cout3.2, Cout4.2, Cout5.2, Cout6.2, Cout9.2, Cvcc1.2, Cvcc2.2, Cvin1.2, J7.2 (Pin_2), J8.2 (Pin_2), Q2.3 (S), Rfbb1.2, Rrenb1.2, Rrt2.2, TP2.1, TP4.1; no longer C2.2, R2.1, U3.10 (PGND), U3.16 (VCCX), U3.7 (AGND)
- net SCL: now also J8.5 (Pin_5)
- net SDA: now also J8.4 (Pin_4)
- net LO: now reaches U3.11 (LO)
- net LO: now also Q2.2 (G)
- net SW: now reaches U3.14 (SW)
- net SW: now also Cboot1.2, Lout1.1, Q1.3 (S), Q2.1 (D)
- net at U2.13 (RBOOT), U2.14 (CBOOT): now also Cboot2.1
- net at U2.10 (SW): now also Cboot2.2, Lout2.1
- net VCC: now reaches U3.9 (VCC)
- net VCC: now also Cvcc1.1
- net at U2.4 (FB): now also Cff1.1, Rfbb1.1, Rfbt1.2
- net ISNS_P: now reaches U3.20 (ISNS+)
- net ISNS_P: now also Lout1.2, Rs1.1
- net at U2.2 (VCC): now also Cvcc2.1; no longer C2.1
- net at U2.5 (PGOOD): now also Rpg1.2
- net at U2.6 (RT): now also Rrt2.1; no longer R2.2
- net at U2.7 (EN/SYNC): now also Rent1.2, Rrenb1.1
- net EXTCOMP: now reaches U3.5 (EXTCOMP)
- net EXTCOMP: now also Chf1.2, Rcomp1.2
- net HO: now reaches U3.13 (HO)
- net HO: now also Q1.2 (G)
- net at U3.17 (PG/SYNCOUT): now also R3.2
- net VDDA: now reaches U3.8 (VDDA)
- net VDDA: now also Cvdda1.1, Rfb1.2; no longer U3.18 (PFM/SYNC)
- net CBOOT_SW: now reaches U3.15 (CBOOT)
- net CBOOT_SW: now also Cboot1.1
- net CNFG: now reaches U3.3 (CNFG)
- net CNFG: now also Rcnfg1.1
- net RT: now reaches U3.4 (RT)
- net RT: now also Rrt1.1
- net FB: now reaches U3.6 (FB)
- net FB: now also Rfb1.1
- net MOSI: now reaches U5.12 (IO8)
- net MOSI: now also J7.7 (Pin_7)
- net SCK: now reaches U5.17 (IO9)
- net SCK: now also J7.5 (Pin_5)
- net CS: now reaches U5.18 (IO10)
- net CS: now also J7.8 (Pin_8)
- net MISO: now reaches U5.19 (IO11)
- net MISO: now also J7.6 (Pin_6)
- net RST: now reaches U5.20 (IO12)
- net RST: now also J7.9 (Pin_9)
- net DINT: now reaches U5.21 (IO13)
- net DINT: now also J7.11 (Pin_11)
- net +5V_Jump renamed +5V
- net +5V: now also U3.16 (VCCX), C1.1, C4.1, JP1.2 (C)
- net +5V_input renamed +5V_IN
- net +5V_IN: now also Cout5.1, Cout6.1, JP1.3 (B), Lout2.2, Rfbt1.1, Rff1.1, Rpg1.1
- net +5V_usb renamed +5V_USB
- net +5V_USB: now also JP1.1 (A)
- net +VBUS renamed +24V
- net +24V: now also Cin-hf1.1, Cin-hf2.1, Cin1.1, Cin2.1, Cin3.1, Cin4.1, Cin5.1, Cin6.1, Cin7.1, Cin8.1, Cinblk1.1, Cvin1.1, Q1.1 (D), Rent1.1, Ruv1.1, TP1.1; no longer C5.1, C8.1, U3.19 (EN)
- net Data+ renamed USB_DM
- net USB_DM: now also C8.1, J2.A7 (D-), J2.B7 (D-); no longer J2.A6 (D+), J2.B6 (D+)
- net Data- renamed USB_DP
- net USB_DP: now also J2.A6 (D+), J2.B6 (D+), C7.1; no longer J2.A7 (D-), J2.B7 (D-)
- net Heater Vcc 1 renamed +12V
- net +12V: now also Cout1.1, Cout2.1, Cout3.1, Cout4.1, Cout9.1, J5.1 (Pin_1), J5.2 (Pin_2), R3.1, Rs1.2, TP3.1
- net Heater_1 renamed Heater1-
- net Heater1-: now also J4.1 (Pin_1)
- net Heater_2 renamed Heater2-
- net Heater2-: now also J4.2 (Pin_2)
- net gpio6 renamed GPIO6
- net gpio7 renamed GPIO7
- new net: Cff1.2, Rff1.2
- new net: Ccomp1.2, Rcomp1.1
- new net AGND: Ccomp1.1, Chf1.1, Cvdda1.2, Rcnfg1.2, Rrt1.2, Ruv2.2, U3.10 (PGND), U3.7 (AGND)
- new net EN: Ruv1.2, Ruv2.1, U3.19 (EN)
- no-connect marks 35 -> 36
Other:
- note added: "+12 BUCK CONVERTER"
- note added: "+5 BUCK CONVERTER"
- note added: "3.3 VOLTAGE REGULATOR"
- note added: "BUTTONS"
- note added: "ESP32-S3-WROOM"
- note added: "HEATER SWITCH"
- note added: "Heater Pins"
- note added: "Heater1+"
- note added: "Heater2+"
- note added: "LCD Display"
- note added: "POWER INPUT"
- note added: "USB-C"
- note added: "temp/humity sensors"
- note removed: "12V Buck"
- note removed: "Power Input"
- moved on the sheet: C27, C28, C32, D1, D3, F1, J1, J2, Q5, Q6, R18, R23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

Commit message: pcb updates
Parts:
- removed Ccomp1: 3.3nF, Capacitor_SMD:C_0402_1005Metric_Pad0.74x0.62mm_HandSolder, symbol Device:C
- removed Chf1: 33pF, Capacitor_SMD:C_0402_1005Metric_Pad0.74x0.62mm_HandSolder, symbol Device:C
- removed Cin4: 10uF, Capacitor_SMD:C_1210_3225Metric_Pad1.33x2.70mm_HandSolder, symbol Device:C
- removed Cin7: .1uF, Capacitor_SMD:C_0402_1005Metric_Pad0.74x0.62mm_HandSolder, symbol Device:C
- removed Cout4: 22uF, Capacitor_SMD:C_1210_3225Metric_Pad1.33x2.70mm_HandSolder, symbol Device:C
- removed Cvcc1: 2.2uF, Capacitor_SMD:C_0603_1608Metric_Pad1.08x0.95mm_HandSolder, symbol Device:C
- removed Cvin1: 22nF, Capacitor_SMD:C_0603_1608Metric_Pad1.08x0.95mm_HandSolder, symbol Device:C
- removed Q1, Q2: NMOS, footprints:TRANS_CSD18512Q5B, symbol Simulation_SPICE:NMOS
- removed R3: 100k, Resistor_SMD:R_0402_1005Metric_Pad0.72x0.64mm_HandSolder, symbol Device:R
- removed Rfb1: 48.7k, Resistor_SMD:R_0402_1005Metric_Pad0.72x0.64mm_HandSolder, symbol Device:R
- removed Ruv1: 200k, Resistor_SMD:R_0402_1005Metric_Pad0.72x0.64mm_HandSolder, symbol Device:R
- removed Ruv2: 9.53k, Resistor_SMD:R_0402_1005Metric_Pad0.72x0.64mm_HandSolder, symbol Device:R
- removed U1: TPD4E02B04DQA, Package_SON:USON-10_2.5x1.0mm_P0.5mm, symbol Power_Protection:TPD4E02B04DQA
- added Cvdda1: .1uf, Capacitor_SMD:C_0402_1005Metric_Pad0.74x0.62mm_HandSolder, symbol Device:C
- added D4, D5, D6: LESD5D5.0CT1G, footprints:TVS_LESD5D5.0CT1G, symbol BreadBoard:LESD5D5.0CT1G
- added Q1, Q3: CSD18512Q5B, footprints:TRANS_CSD18512Q5B, symbol BreadBoard:CSD18512Q5B
- added Rpg2: 100k, Resistor_SMD:R_0201_0603Metric_Pad0.64x0.40mm_HandSolder, symbol Device:R
- added Rvdda1: 47.5k, Resistor_SMD:R_0201_0603Metric_Pad0.64x0.40mm_HandSolder, symbol Device:R
- added TP5: 5out, TestPoint:TestPoint_Keystone_5019_Miniature, symbol Connector:TestPoint
- added TP6: 5v_out, TestPoint:TestPoint_Keystone_5019_Miniature, symbol Connector:TestPoint
- added TP7: 3.3V, TestPoint:TestPoint_Keystone_5019_Miniature, symbol Connector:TestPoint
- Cin1: value 10uF -> 4.7uF
- Cin2, Cin3: value 10uF -> 4.7
- Cvcc1: renamed from Cvdda1; value 0.47uF -> 2.2uF
- F1: footprint footprints:FUSC6125X279N -> footprints:FUS_CB_3216TD
- J7: footprint Connector_PinHeader_2.54mm:PinHeader_1x15_P2.54mm_Vertical -> Connector_PinSocket_1.00mm:PinSocket_1x15_P1.00mm_Vertical
- J8: footprint Connector_PinHeader_2.54mm:PinHeader_1x05_P2.54mm_Vertical -> Connector_PinSocket_1.00mm:PinSocket_1x05_P1.00mm_Vertical
- Lout2: footprint footprints:IND_NS12565T100MNV_TAY -> footprints:WSR-L
- Rcnfg1: value 29.4k -> 41.2k
- Rcomp1: value 11.8k -> 10k; footprint Resistor_SMD:R_0402_1005Metric_Pad0.72x0.64mm_HandSolder -> Resistor_SMD:R_0201_0603Metric_Pad0.64x0.40mm_HandSolder
- Rrt1: value 54.9k -> 51.1k
- TP2: value TestPoint:TestPoint_Keystone_5019_Miniature -> +24_gnd; footprint (none) -> TestPoint:TestPoint_Keystone_5019_Miniature
- TP4: value 12V_out_gnd -> gnd
Connections:
- net EN is gone; now on net +24V: U3.19 (EN)
- net +24V: now also Q3.5_8
- net +3.3V: now also TP7.1
- net +5V: no longer U3.16 (VCCX)
- net +5V_IN: now also TP6.1
- net AGND: now also U3.23 (NC), U3.24 (NC), U3.25 (EP), Cvdda1.2; no longer Cvcc1.2, U3.10 (PGND)
- net EXTCOMP: now also Rcomp1.1; no longer Rcomp1.2
- net FB: now also Rvdda1.1
- net GND: now also Cvcc1.2, U3.1 (NC), U3.10 (PGND), U3.16 (VCCX), U3.2 (NC), U3.22 (NC), D4.1, D5.1, D6.1, Q1.1, Q1.2, Q1.3, TP5.1; no longer U3.18 (PFM/SYNC), U3.25 (EP)
- net HO: now also Q3.4
- net LO: now also Q1.4
- net SCL: now also U5.9 (IO16); no longer U5.38 (IO2)
- net SDA: now also U5.8 (IO15); no longer U5.39 (IO1)
- net SW: now also Q1.5_8, Q3.1, Q3.2, Q3.3
- net VCC: now also Cvcc1.1, Rpg2.1
- net VDDA: now also Rcomp1.2, U3.18 (PFM/SYNC), Cvdda1.1, Rvdda1.2; no longer Cvcc1.1
- net at D2.2 (A), J2.A4 (VBUS), J2.A9 (VBUS)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: now also D6.2
- net at U3.17 (PG/SYNCOUT): now also Rpg2.2
- net USB_DM renamed USB_D+
- net USB_D+: now also J2.A6 (D+), J2.B6 (D+), D4.2; no longer J2.A7 (D-), J2.B7 (D-)
- net USB_DP renamed USB_D-
- net USB_D-: now also J2.A7 (D-), J2.B7 (D-), D5.2; no longer J2.A6 (D+), J2.B6 (D+)
Other:
- moved on the sheet: Cin5, Cin6, Cin8, Cvcc1, Rcnfg1, Rrt1, TP1, TP2, TP4
