File: BreadBoard_git/BreadBoard_git.kicad_sch (KiCad schematic)
At the start: 88 parts, among them J1 PD-40, J2 USB_C_Receptacle_USB2.0_14P, J4 Conn_01x02_Pin, J5 Conn_01x02_Pin, J7 Conn_01x15_Pin, J8 Conn_01x05_Pin, Q1 CSD18512Q5B, Q3 CSD18512Q5B, Q5 RQ3E110AJTB, Q6 RQ3E110AJTB, SW1 SKRPADE010, SW2 SKRPADE010, U2 LM61460AANRJRR, U3 LM5148RGYR, U4 AMS1117-3.3, U5 ESP32-S3-WROOM-1

Commit message: updates!
Parts:
- added TP8: gnd, TestPoint:TestPoint_Keystone_5019_Miniature, symbol Connector:TestPoint
Connections:
- net +12V: now also J4.1 (Pin_1); no longer J5.2 (Pin_2)
- net BOOT: now also SW2.2
- net CHIP_PU: now also SW1.2
- net GND: now also SW1.4, SW2.4, TP8.1; no longer Cin1.2, Cin2.2, Cin3.2, Cin5.2, Cin6.2, Cin8.2, Cout1.2, Cout2.2, Cout3.2, Cout9.2, D1.A, J1.2, J1.3, J1.S1 (SHIELD), Q1.1, Q1.2, Q1.3, TP2.1, TP4.1, U3.10 (PGND), U3.16 (VCCX)
- net Heater1-: now also J5.2 (Pin_2); no longer J4.1 (Pin_1)
- new net PGND: Cin1.2, Cin2.2, Cin3.2, Cin5.2, Cin6.2, Cin8.2, Cout1.2, Cout2.2, Cout3.2, Cout9.2, D1.A, J1.2, J1.3, J1.S1 (SHIELD), Q1.1, Q1.2, Q1.3, TP2.1, TP4.1, U3.10 (PGND), U3.16 (VCCX)
- no-connect marks 36 -> 32

Commit message: updates
Parts:
- removed TP1: 24V_in, TestPoint:TestPoint_Keystone_5019_Miniature, symbol Connector:TestPoint
- removed TP2: +24_gnd, TestPoint:TestPoint_Keystone_5019_Miniature, symbol Connector:TestPoint
- removed TP3: 12V_out, TestPoint:TestPoint_Keystone_5019_Miniature, symbol Connector:TestPoint
- removed TP4, TP8: gnd, TestPoint:TestPoint_Keystone_5019_Miniature, symbol Connector:TestPoint
- removed TP5: 5out, TestPoint:TestPoint_Keystone_5019_Miniature, symbol Connector:TestPoint
- removed TP6: 5v_out, TestPoint:TestPoint_Keystone_5019_Miniature, symbol Connector:TestPoint
- removed TP7: 3.3V, TestPoint:TestPoint_Keystone_5019_Miniature, symbol Connector:TestPoint
- added Cinblk2: 10uF, Capacitor_SMD:C_1210_3225Metric_Pad1.33x2.70mm_HandSolder, symbol Device:C
- added J6: Conn_01x08_Socket, Connector_PinSocket_2.54mm:PinSocket_1x08_P2.54mm_Vertical, symbol Connector:Conn_01x08_Socket
- added R3, R5: 4.7k, symbol Device:R
- C1, C2: value 10uF -> 22uF
Connections:
- net +24V: now also Cinblk2.1
- net +3.3V: now also R3.1, R5.1
- net CS: now also U5.20 (IO12); no longer U5.18 (IO10)
- net DINT: now also U5.22 (IO14); no longer U5.21 (IO13)
- net GND: now also Cinblk2.2, J6.8 (Pin_8)
- net MISO: now also U5.18 (IO10); no longer U5.19 (IO11)
- net MOSI: now also U5.19 (IO11); no longer U5.12 (IO8)
- net RST: now also U5.21 (IO13); no longer U5.20 (IO12)
- net SCL: now also R5.2
- net SDA: now also R3.2
- net vbus: now reaches F1.1, J1.1, J1.4
- net GPIO38: now reaches U5.31 (IO38)
- net GPIO38: now also J6.1 (Pin_1)
- net GPIO39: now reaches U5.32 (IO39)
- net GPIO39: now also J6.2 (Pin_2)
- net GPIO40: now reaches U5.33 (IO40)
- net GPIO40: now also R26.1
- net GPIO41: now reaches U5.34 (IO41)
- net GPIO41: now also R25.1
- net GPIO42: now reaches U5.35 (IO42)
- net GPIO42: now also J6.3 (Pin_3)
- net RXDO: now reaches U5.36 (RXD0)
- net RXDO: now also J6.4 (Pin_4)
- net TXD0: now reaches U5.37 (TXD0)
- net TXD0: now also J6.5 (Pin_5)
- net GPIO2: now reaches U5.38 (IO2)
- net GPIO2: now also J6.6 (Pin_6)
- net GPIO1: now reaches U5.39 (IO1)
- net GPIO1: now also J6.7 (Pin_7)
- net GPIO6: no longer names the net of U5.6 (IO6)
- net GPIO6: no longer R25.1
- net GPIO7: no longer names the net of U5.7 (IO7)
- net GPIO7: no longer R26.1
- net HO renamed SW-
- net SW renamed SW+
- no-connect marks 32 -> 24
