File: BreadBoard_git/BreadBoard_git.kicad_pcb (KiCad board)
At the start: 2 copper layers, 105.9 x 45.9 mm, 73 parts, among them J1 PD-40, J2 USB_C_Receptacle_USB2.0_14P, J3 Conn_01x02_Pin, Q3 CSD18512Q5B, Q4 CSD18512Q5B, Q5 RQ3E110AJTB, Q6 RQ3E110AJTB, SW1 SKRPADE010, SW2 SKRPADE010, U1 TPD4E02B04DQA, U2 LM61460AANRJRR, U3 LM5148RGYR, U4 AMS1117-3.3, U5 ESP32-S3-WROOM-1

Commit message: update!
Parts:
- removed C10: CL05C821JB5NNNC, footprints:CAP_CL05_SAM-L
- removed C11: C0402C300J5GACTU, footprints:CAPC10555_55N_KEM-L
- removed C12, C23, C24, C25: MSAST21GBB5106MTNA01, footprints:CAPC2012X145N
- removed C13, C35: GRM32ER71H475KA88L, footprints:CAPC3225X270N
- removed C14: GRM155R71A104KA01D, footprints:CAPC1005X55N
- removed C15: GRM033R61A104KE15D, footprints:CAPC0603X33N
- removed C16: 10uF, footprints:RC0603N_YAG-L
- removed C17: GRM155R71A104KA01D, footprints:G-155_MUR-L
- removed C18, C21: 100nF, footprints:RC0603N_YAG-L
- removed C19: CC0805JRNPO9BN120, footprints:CAP_CC0805_YAG-L
- removed C20: GRM31CR61A107MEA8K, footprints:CAPC3216X190N
- removed C22: 22uF, footprints:RC0603N_YAG-L
- removed C26, C34: 0402B104K500HI, Capacitor_SMD:C_0402_1005Metric_Pad0.74x0.62mm_HandSolder
- removed C9: GRM188R71A225KE15D, footprints:G-188_MUR-L
- removed J3: Conn_01x02_Pin, Connector_PinHeader_1.00mm:PinHeader_1x02_P1.00mm_Vertical
- removed JP1: Jumper_3_Open, Connector_Samtec_HPM_THT:Samtec_HPM-03-01-x-S_Straight_1x03_Pitch5.08mm
- removed L1: WE-XHMI_5050, footprints:WE-XHMI_5050
- removed L2: CDEP63MENP-R68MC, footprints:IND_CDEP63MENP-R68MC_SUM-L
- removed Q3, Q4: CSD18512Q5B, footprints:TRANS_CSD18512Q5B
- removed Q5, Q6: RQ3E110AJTB, footprints:HSMT8_ROM-L
- removed R11: RC0603FR-0740K2L, footprints:RC0603N_YAG-L
- removed R14, R8: CRCW0402100KFKED, footprints:RES_CRCW_0402_VIS-L
- removed R15: RC0603FR-0724K9L, footprints:RC0603N_YAG-L
- removed R16: RC0603FR-079K53L, footprints:RC0603N_YAG-L
- removed R17: CRCW04021K00FKED, footprints:RESC1005X40N
- removed R19: WSR23L000FEA, footprints:WSR-L
- removed R25, R26: 47, Resistor_SMD:R_0201_0603Metric_Pad0.64x0.40mm_HandSolder
- removed R27, R28: 100k, Resistor_SMD:R_0201_0603Metric_Pad0.64x0.40mm_HandSolder
- removed R5: CRCW0603100KFKEA, footprints:RES_CRCW_0603_VIS-L
- removed R7: CRCW04024K87FKED, footprints:RES_CRCW_0402-L
- removed R9: 10k, Resistor_SMD:R_0201_0603Metric
- added Cboot1: 0.1 µF, Resistor_SMD:R_0402_1005Metric_Pad0.72x0.64mm_HandSolder, F.Cu at (100.2, 81.2)
- added Cboot2: .1uF, Capacitor_SMD:C_0201_0603Metric_Pad0.64x0.40mm_HandSolder, F.Cu at (108.2, 49.0)
- added Ccomp1: 3.3nF, Capacitor_SMD:C_0402_1005Metric_Pad0.74x0.62mm_HandSolder, F.Cu at (94.2, 90.4)
- added Cff1: 33pF, Capacitor_SMD:C_0201_0603Metric_Pad0.64x0.40mm_HandSolder, F.Cu at (101.2, 57.8)
- added Chf1: 33pF, Capacitor_SMD:C_0402_1005Metric_Pad0.74x0.62mm_HandSolder, F.Cu at (95.2, 90.4)
- added Cin-hf1: 220nF, Capacitor_SMD:C_0603_1608Metric_Pad1.08x0.95mm_HandSolder, F.Cu at (112.0, 60.0)
- added Cin-hf2: 220nF, Capacitor_SMD:C_0603_1608Metric_Pad1.08x0.95mm_HandSolder, F.Cu at (112.1, 48.6)
- added Cin1: 10uF, Capacitor_SMD:C_1210_3225Metric_Pad1.33x2.70mm_HandSolder, F.Cu at (109.0, 84.6)
- added Cin2: 10uF, Capacitor_SMD:C_1210_3225Metric_Pad1.33x2.70mm_HandSolder, F.Cu at (107.6, 89.0)
- added Cin3: 10uF, Capacitor_SMD:C_1210_3225Metric_Pad1.33x2.70mm_HandSolder, F.Cu at (107.6, 92.2)
- added Cin4: 10uF, Capacitor_SMD:C_1210_3225Metric_Pad1.33x2.70mm_HandSolder, F.Cu at (107.6, 95.4)
- added Cin5: .1uF, Capacitor_SMD:C_0402_1005Metric_Pad0.74x0.62mm_HandSolder, F.Cu at (111.2, 98.1)
- added Cin6: .1uF, Capacitor_SMD:C_0402_1005Metric_Pad0.74x0.62mm_HandSolder, F.Cu at (116.0, 98.0)
- added Cin7: .1uF, Capacitor_SMD:C_0402_1005Metric_Pad0.74x0.62mm_HandSolder, F.Cu at (114.4, 98.0)
- added Cin8: .1uF, Capacitor_SMD:C_0402_1005Metric_Pad0.74x0.62mm_HandSolder, F.Cu at (112.8, 98.0)
- added Cinblk1: 10uF, Capacitor_SMD:C_1210_3225Metric_Pad1.33x2.70mm_HandSolder, F.Cu at (114.0, 65.8)
- added Cout1: 22uF, Capacitor_SMD:C_1210_3225Metric_Pad1.33x2.70mm_HandSolder, F.Cu at (128.4, 83.6)
- added Cout2: 22uF, Capacitor_SMD:C_1210_3225Metric_Pad1.33x2.70mm_HandSolder, F.Cu at (128.4, 80.2)
- added Cout3: 22uF, Capacitor_SMD:C_1210_3225Metric_Pad1.33x2.70mm_HandSolder, F.Cu at (128.4, 94.8)
- added Cout4: 22uF, Capacitor_SMD:C_1210_3225Metric_Pad1.33x2.70mm_HandSolder, F.Cu at (128.4, 98.0)
- added Cout5: 47uf, Capacitor_SMD:C_1210_3225Metric_Pad1.33x2.70mm_HandSolder, F.Cu at (129.4, 42.6)
- added Cout6: 47uF, Capacitor_SMD:C_1210_3225Metric_Pad1.33x2.70mm_HandSolder, F.Cu at (128.4, 65.2)
- added Cout9: .1uF, Capacitor_SMD:C_0402_1005Metric_Pad0.74x0.62mm_HandSolder, F.Cu at (140.2, 89.2)
- added Cvcc1: 2.2uF, Capacitor_SMD:C_0603_1608Metric_Pad1.08x0.95mm_HandSolder, F.Cu at (101.2, 88.4)
- added Cvcc2: 1uF, Capacitor_SMD:C_0603_1608Metric_Pad1.08x0.95mm_HandSolder, F.Cu at (105.2, 53.8)
- added Cvdda1: 0.47uF, Capacitor_SMD:C_0402_1005Metric_Pad0.74x0.62mm_HandSolder, F.Cu at (99.0, 88.8)
- added Cvin1: 22nF, Capacitor_SMD:C_0603_1608Metric_Pad1.08x0.95mm_HandSolder, F.Cu at (101.8, 78.3)
- added Lout1: 4.7u, footprints:WSR-L, F.Cu at (124.6, 89.4)
- added Lout2: 22uF, footprints:IND_NS12565T100MNV_TAY, F.Cu at (116.4, 53.8)
- added Q1: NMOS, footprints:TRANS_CSD18512Q5B, F.Cu at (113.6, 85.2)
- added Q2: NMOS, footprints:TRANS_CSD18512Q5B, F.Cu at (113.6, 92.8)
- added Rcnfg1: 29.4k, Resistor_SMD:R_0402_1005Metric_Pad0.72x0.64mm_HandSolder, F.Cu at (92.4, 87.8)
- added Rcomp1: 11.8k, Resistor_SMD:R_0402_1005Metric_Pad0.72x0.64mm_HandSolder, F.Cu at (94.8, 88.4)
- added Rent1: 255k, Resistor_SMD:R_0603_1608Metric_Pad0.98x0.95mm_HandSolder, F.Cu at (106.3, 69.4)
- added Rfb1: 48.7k, Resistor_SMD:R_0402_1005Metric_Pad0.72x0.64mm_HandSolder, F.Cu at (97.2, 88.4)
- added Rfbb1: 24.9k, Resistor_SMD:R_0603_1608Metric_Pad0.98x0.95mm_HandSolder, F.Cu at (102.8, 56.0)
- added Rfbt1: 100k, Resistor_SMD:R_0603_1608Metric_Pad0.98x0.95mm_HandSolder, F.Cu at (99.4, 58.0)
- added Rff1: 1k, Resistor_SMD:R_0603_1608Metric_Pad0.98x0.95mm_HandSolder, F.Cu at (100.2, 61.6)
- added Rpg1: 100k, Resistor_SMD:R_0603_1608Metric_Pad0.98x0.95mm_HandSolder, F.Cu at (99.3, 69.1)
- added Rrenb1: 100k, Resistor_SMD:R_0603_1608Metric_Pad0.98x0.95mm_HandSolder, F.Cu at (106.4, 66.2)
- added Rrt1: 54.9k, Resistor_SMD:R_0402_1005Metric_Pad0.72x0.64mm_HandSolder, F.Cu at (92.4, 88.8)
- added Rrt2: 33.2k, Resistor_SMD:R_0603_1608Metric_Pad0.98x0.95mm_HandSolder, F.Cu at (107.2, 59.8)
- added Rs1: 4.3m, Resistor_SMD:R_0508_1220Metric_Pad1.12x2.15mm_HandSolder, F.Cu at (132.5, 89.4)
- added Ruv1: 200k, Resistor_SMD:R_0402_1005Metric_Pad0.72x0.64mm_HandSolder, F.Cu at (96.8, 81.2)
- added Ruv2: 9.53k, Resistor_SMD:R_0402_1005Metric_Pad0.72x0.64mm_HandSolder, F.Cu at (91.2, 81.8)
- added TP1: 24V_in, TestPoint:TestPoint_Keystone_5019_Miniature, F.Cu at (79.8, 80.8)
- added TP2: +24_gnd, TestPoint:TestPoint_Keystone_5019_Miniature, F.Cu at (148.2, 91.0)
- added TP3: 12V_out, TestPoint:TestPoint_Keystone_5019_Miniature, F.Cu at (147.4, 79.4)
- added TP4: gnd, TestPoint:TestPoint_Keystone_5019_Miniature, F.Cu at (79.2, 91.8)
- added TP5: 5out, TestPoint:TestPoint_Keystone_5019_Miniature, F.Cu at (137.4, 58.6)
- added TP6: 5v_out, TestPoint:TestPoint_Keystone_5019_Miniature, F.Cu at (137.2, 49.6)
- added TP7: 3.3V, TestPoint:TestPoint_Keystone_5019_Miniature, F.Cu at (167.6, 53.4)
- C1: value C2012X6S1H155K125AB -> 10uF; footprint footprints:CAP_2012_TDK-L -> Capacitor_SMD:C_0603_1608Metric_Pad1.08x0.95mm_HandSolder
- C2: value GRM188R60J105KA01D -> 10uF; footprint footprints:G-188_MUR-L -> Capacitor_SMD:C_0603_1608Metric_Pad1.08x0.95mm_HandSolder
- C27: footprint footprints:G-155_MUR-L -> Capacitor_SMD:C_0805_2012Metric_Pad1.18x1.45mm_HandSolder
- C28: value 100nF -> 0u1F; footprint footprints:CAPC0603X33N -> Capacitor_SMD:C_0603_1608Metric_Pad1.08x0.95mm_HandSolder
- C3, C4, C6: value C2012X6S1H155K125AB -> 0u1F; footprint footprints:CAP_2012_TDK-L -> Capacitor_SMD:C_0603_1608Metric_Pad1.08x0.95mm_HandSolder
- C32: footprint footprints:CAPC0603X33N -> Capacitor_SMD:C_0603_1608Metric_Pad1.08x0.95mm_HandSolder
- C5: value C1005X5R1V474K050BC -> 0u1F; footprint footprints:CAPC1005X55N -> Capacitor_SMD:C_0603_1608Metric_Pad1.08x0.95mm_HandSolder
- C7: value GRM155R71A104KA01D -> 22pF; footprint footprints:G-155_MUR-L -> Capacitor_SMD:C_0402_1005Metric_Pad0.74x0.62mm_HandSolder
- C8: value C1005X5R1V474K050BC -> 22pF; footprint footprints:CAPC1005X55N -> Capacitor_SMD:C_0402_1005Metric_Pad0.74x0.62mm_HandSolder
- D2: footprint Diode_SMD:D_SOD-523 -> Diode_SMD:D_0603_1608Metric_Pad1.05x0.95mm_HandSolder
- F1: value TR/3216TD12-R -> 0680L6300-05; footprint footprints:FUS_CB_3216TD -> footprints:FUSC6125X279N
- R1, R23: footprint Resistor_SMD:R_0201_0603Metric -> Resistor_SMD:R_0603_1608Metric_Pad0.98x0.95mm_HandSolder
- R18: value 150 -> 75
- R2: value GRM188R60J105KA01D -> 10k; footprint footprints:RESC2012X50N -> Resistor_SMD:R_0603_1608Metric_Pad0.98x0.95mm_HandSolder
- R3: value CRCW060347K5FKEA -> 100k; footprint footprints:RES_CRCW_0603-L -> Resistor_SMD:R_0402_1005Metric_Pad0.72x0.64mm_HandSolder
- moved R1 147.6 mm to (148.7, 64.8)
- moved SW1 143.3 mm to (154.3, 63.8)
- moved SW2 143.3 mm to (154.3, 70.4)
- moved R3 126.4 mm to (97.8, 81.2), turned to -90 degrees
- moved C8 116.1 mm to (174.3, 42.4), turned to -90 degrees
- moved C2 102.6 mm to (155.9, 45.1), turned to 90 degrees
- moved C5 83.8 mm to (148.6, 63.0), turned to 180 degrees
- moved R2 83.7 mm to (148.6, 69.2)
- moved U3 82.7 mm to (97.0, 85.0), turned to 90 degrees
- moved C3 82.0 mm to (157.7, 45.1), turned to 90 degrees
- moved C4 80.8 mm to (157.7, 49.1), turned to -90 degrees
- moved U2 79.4 mm to (109.5, 54.0)
- moved C1 75.0 mm to (155.7, 49.1), turned to -90 degrees
- moved C7 72.1 mm to (176.3, 42.4), turned to -90 degrees
- moved F1 68.3 mm to (90.2, 56.8), turned to 90 degrees
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Connections:
- net +5V_usb renamed +5V_USB
- C1 pad 1: GND -> +5V
- C1 pad 2: +VBUS -> GND
- C2 pad 1: Net-(U2-VCC) -> GND
- C2 pad 2: GND -> +3.3V
- C3 pad 1: GND -> +3.3V
- C3 pad 2: +VBUS -> GND
- C32 pad 1: CHIP_PU -> /CHIP_PU
- C4 pad 1: GND -> +5V
- C4 pad 2: +VBUS -> GND
- C5 pad 1: +VBUS -> /CHIP_PU
- C6 pad 1: GND -> /BOOT
- C6 pad 2: +VBUS -> GND
- C7 pad 1: GND -> /USB_DP
- C7 pad 2: Net-(U3-PFM/SYNC) -> GND
- C8 pad 1: +VBUS -> /USB_DM
- D1 pad C: +VBUS -> +24V
- F1 pad 2: +VBUS -> +24V
- J2 pad A6: Data+ -> /USB_DP
- J2 pad A7: Data- -> /USB_DM
- J2 pad B6: Data+ -> /USB_DP
- J2 pad B7: Data- -> /USB_DM
- R1 pad 2: CHIP_PU -> /CHIP_PU
- R2 pad 1: GND -> +3.3V
- R2 pad 2: Net-(U2-RT) -> /BOOT
- R23 pad 2: CHIP_PU -> /CHIP_PU
- R3 pad 1: Net-(U3-PFM/SYNC) -> +12V
- R3 pad 2: Net-(U3-FB) -> Net-(U3-PG/SYNCOUT)
- SW1 pad 1: CHIP_PU -> /CHIP_PU
- SW2 pad 1: BOOT -> /BOOT
- U1 pad 4: Data+ -> /USB_DM
- U1 pad 5: Data- -> /USB_DP
- U2 pad 1: +5V_input -> +5V_IN
- U2 pad 12: +VBUS -> +24V
- U2 pad 7: unconnected-(U2-EN/SYNC-Pad7) -> Net-(U2-EN/SYNC)
- U2 pad 8: +VBUS -> +24V
- U3 pad 10: GND -> AGND
- U3 pad 11: Net-(U3-LO) -> /LO
- U3 pad 12: +VBUS -> +24V
- U3 pad 13: Net-(U3-HO) -> /HO
- U3 pad 14: Net-(U3-SW) -> /SW
- U3 pad 15: Net-(U3-CBOOT) -> /CBOOT_SW
- U3 pad 16: GND -> +5V
- U3 pad 18: Net-(U3-PFM/SYNC) -> GND
- U3 pad 19: +VBUS -> /EN
- U3 pad 20: Net-(U3-ISNS+) -> /ISNS_P
- U3 pad 21: Heater Vcc 1 -> +12V
- U3 pad 3: Net-(U3-CNFG) -> /CNFG
- U3 pad 4: Net-(U3-RT) -> /RT
- U3 pad 5: Net-(U3-EXTCOMP) -> /EXTCOMP
- U3 pad 6: Net-(U3-FB) -> /FB
- U3 pad 7: GND -> AGND
- U3 pad 8: Net-(U3-PFM/SYNC) -> /VDDA
- U3 pad 9: Net-(U3-VCC) -> /VCC
- U4 pad 3: +5V_Jump -> +5V
- U5 pad 12: unconnected-(U5-IO8-Pad12) -> /MOSI
- U5 pad 13: Data- -> /USB_DP
- U5 pad 14: Data+ -> /USB_DM
- U5 pad 17: unconnected-(U5-IO9-Pad17) -> /SCK
- U5 pad 18: unconnected-(U5-IO10-Pad18) -> /CS
- U5 pad 19: unconnected-(U5-IO11-Pad19) -> /MISO
- U5 pad 20: unconnected-(U5-IO12-Pad20) -> /RST
- U5 pad 21: unconnected-(U5-IO13-Pad21) -> /DINT
- U5 pad 27: BOOT -> /BOOT
- U5 pad 3: CHIP_PU -> /CHIP_PU
- U5 pad 38: SCL -> /SCL
- U5 pad 39: SDA -> /SDA
- U5 pad 6: gpio6 -> /GPIO6
- U5 pad 7: gpio7 -> /GPIO7
Routing:
- net (no net): vias 0 -> 1
- added copper zone on In1.Cu, net GND
Other:
- board size 105.9 x 45.9 mm -> 119 x 62.6 mm
- copper layers 2 -> 4

Commit message: pcb updates
Parts:
- removed Ccomp1: 3.3nF, Capacitor_SMD:C_0402_1005Metric_Pad0.74x0.62mm_HandSolder
- removed Chf1: 33pF, Capacitor_SMD:C_0402_1005Metric_Pad0.74x0.62mm_HandSolder
- removed Cin4: 10uF, Capacitor_SMD:C_1210_3225Metric_Pad1.33x2.70mm_HandSolder
- removed Cin7: .1uF, Capacitor_SMD:C_0402_1005Metric_Pad0.74x0.62mm_HandSolder
- removed Cout4: 22uF, Capacitor_SMD:C_1210_3225Metric_Pad1.33x2.70mm_HandSolder
- removed Cvin1: 22nF, Capacitor_SMD:C_0603_1608Metric_Pad1.08x0.95mm_HandSolder
- removed Q2: NMOS, footprints:TRANS_CSD18512Q5B
- removed R3: 100k, Resistor_SMD:R_0402_1005Metric_Pad0.72x0.64mm_HandSolder
- removed Rfb1: 48.7k, Resistor_SMD:R_0402_1005Metric_Pad0.72x0.64mm_HandSolder
- removed Ruv1: 200k, Resistor_SMD:R_0402_1005Metric_Pad0.72x0.64mm_HandSolder
- removed Ruv2: 9.53k, Resistor_SMD:R_0402_1005Metric_Pad0.72x0.64mm_HandSolder
- removed U1: TPD4E02B04DQA, Package_SON:USON-10_2.5x1.0mm_P0.5mm
- added D4: LESD5D5.0CT1G, footprints:TVS_LESD5D5.0CT1G, F.Cu at (166.6, 89.8)
- added D5: LESD5D5.0CT1G, footprints:TVS_LESD5D5.0CT1G, F.Cu at (164.8, 89.8)
- added D6: LESD5D5.0CT1G, footprints:TVS_LESD5D5.0CT1G, F.Cu at (170.0, 90.0)
- added J4: Conn_01x02_Pin, Connector_PinHeader_2.54mm:PinHeader_1x02_P2.54mm_Vertical, F.Cu at (137.2, 147.5)
- added J5: Conn_01x02_Pin, Connector_PinHeader_2.54mm:PinHeader_1x02_P2.54mm_Vertical, F.Cu at (141.8, 147.5)
- added J7: Conn_01x15_Pin, Connector_PinSocket_1.00mm:PinSocket_1x15_P1.00mm_Vertical, F.Cu at (171.0, 61.2)
- added J8: Conn_01x05_Pin, Connector_PinSocket_1.00mm:PinSocket_1x05_P1.00mm_Vertical, F.Cu at (181.2, 40.8)
- added JP1: Jumper_3_Bridged12, Connector_PinHeader_2.54mm:PinHeader_1x03_P2.54mm_Vertical, F.Cu at (155.3, 56.0)
- added Q3: CSD18512Q5B, footprints:TRANS_CSD18512Q5B, F.Cu at (113.6, 92.4)
- added Q5: RQ3E110AJTB, footprints:HSMT8_ROM-L, F.Cu at (142.5, 137.8)
- added Q6: RQ3E110AJTB, footprints:HSMT8_ROM-L, F.Cu at (142.5, 142.6)
- added R25: 47, Resistor_SMD:R_0603_1608Metric_Pad0.98x0.95mm_HandSolder, F.Cu at (132.7, 136.8)
- added R26: 47, Resistor_SMD:R_0603_1608Metric_Pad0.98x0.95mm_HandSolder, F.Cu at (132.7, 139.3)
- added R27: 100k, Resistor_SMD:R_0603_1608Metric_Pad0.98x0.95mm_HandSolder, F.Cu at (132.7, 141.8)
- added R28: 100k, Resistor_SMD:R_0603_1608Metric_Pad0.98x0.95mm_HandSolder, F.Cu at (132.7, 144.3)
- added Rpg2: 100k, Resistor_SMD:R_0201_0603Metric_Pad0.64x0.40mm_HandSolder, F.Cu at (98.0, 82.2)
- added Rvdda1: 47.5k, Resistor_SMD:R_0201_0603Metric_Pad0.64x0.40mm_HandSolder, F.Cu at (97.2, 88.2)
- Cin1: value 10uF -> 4.7uF
- Cin2, Cin3: value 10uF -> 4.7
- Cvcc1: footprint Capacitor_SMD:C_0603_1608Metric_Pad1.08x0.95mm_HandSolder -> Capacitor_SMD:C_0402_1005Metric_Pad0.74x0.62mm_HandSolder
- Cvdda1: value 0.47uF -> .1uf
- F1: footprint footprints:FUSC6125X279N -> footprints:FUS_CB_3216TD
- Lout2: footprint footprints:IND_NS12565T100MNV_TAY -> footprints:WSR-L
- Q1: value NMOS -> CSD18512Q5B
- Rcnfg1: value 29.4k -> 41.2k
- Rcomp1: value 11.8k -> 10k; footprint Resistor_SMD:R_0402_1005Metric_Pad0.72x0.64mm_HandSolder -> Resistor_SMD:R_0201_0603Metric_Pad0.64x0.40mm_HandSolder
- Rrt1: value 54.9k -> 51.1k
- moved C8 51.1 mm to (159.2, 91.2), turned to 180 degrees
- moved C7 50.6 mm to (159.2, 90.0), turned to 180 degrees
- moved C27 14.4 mm to (191.7, 54.8)
- moved C32 14.4 mm to (186.2, 57.0)
- moved C28 14.4 mm to (191.4, 57.2)
- moved U5 14.4 mm to (187.0, 68.0)
- moved R23 12.3 mm to (187.2, 54.2)
- moved D2 10.2 mm to (172.5, 89.0), turned to -90 degrees
- moved R6 8.83 mm to (173.0, 96.3), turned to -90 degrees
- moved J2 8.59 mm to (165.9, 97.0)
- moved R4 8.33 mm to (174.5, 95.8), turned to -90 degrees
- moved TP2 6.94 mm to (143.0, 95.6)
- moved TP3 5.81 mm to (143.0, 83.2)
- moved Cout9 2.82 mm to (143.0, 88.8)
- moved Rfbb1 1.48 mm to (104.3, 56.0)
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Connections:
- C7 pad 1: /USB_DP -> /USB_D-
- C8 pad 1: /USB_DM -> /USB_D+
- Cin1 pad 2: GND -> PGND
- Cin2 pad 2: GND -> PGND
- Cin3 pad 2: GND -> PGND
- Cin5 pad 2: GND -> PGND
- Cin6 pad 2: GND -> PGND
- Cin8 pad 2: GND -> PGND
- J2 pad A6: /USB_DP -> /USB_D+
- J2 pad A7: /USB_DM -> /USB_D-
- J2 pad B6: /USB_DP -> /USB_D+
- J2 pad B7: /USB_DM -> /USB_D-
- Q1 pad 1: +24V -> PGND
- Q1 pad 2: /HO -> PGND
- Q1 pad 3: /SW -> PGND
- Q1 pad 4: (no net) -> /LO
- Q1 pad 5_8: (no net) -> /SW
- Rcomp1 pad 1: Net-(Ccomp1-Pad2) -> /EXTCOMP
- Rcomp1 pad 2: /EXTCOMP -> /VDDA
- TP2 pad 1: GND -> PGND
- U3 pad 1: unconnected-(U3-NC-Pad1) -> GND
- U3 pad 10: AGND -> PGND
- U3 pad 16: +5V -> PGND
- U3 pad 18: GND -> /VDDA
- U3 pad 19: /EN -> +24V
- U3 pad 2: unconnected-(U3-NC-Pad2) -> GND
- U3 pad 22: unconnected-(U3-NC-Pad22) -> GND
- U3 pad 23: unconnected-(U3-NC-Pad23) -> AGND
- U3 pad 24: unconnected-(U3-NC-Pad24) -> AGND
- U3 pad 25: GND -> AGND
- U5 pad 13: /USB_DP -> /USB_D-
- U5 pad 14: /USB_DM -> /USB_D+
- U5 pad 38: /SCL -> unconnected-(U5-IO2-Pad38)
- U5 pad 39: /SDA -> unconnected-(U5-IO1-Pad39)
- U5 pad 8: unconnected-(U5-IO15-Pad8) -> /SDA
- U5 pad 9: unconnected-(U5-IO16-Pad9) -> /SCL
Routing:
- net /USB_D+: track 0.00 -> 55.0 mm, vias 0 -> 2
- net /USB_D-: track 0.00 -> 54.2 mm
- net GND: track 0.00 -> 25.4 mm, vias 0 -> 20
- net /SDA: track 0.00 -> 20.6 mm
- net /SCL: track 0.00 -> 20.5 mm
- net Net-(D2-A): track 0.00 -> 18.7 mm, vias 0 -> 2
- net /SW: track 0.00 -> 17.4 mm, vias 0 -> 2
- net /CS: track 0.00 -> 14.4 mm, vias 0 -> 2
- net /MOSI: track 0.00 -> 14.1 mm, vias 0 -> 2
- net +24V: track 0.00 -> 13.0 mm, vias 0 -> 11
- net /VCC: track 0.00 -> 11.0 mm, vias 0 -> 2
- net Net-(J2-CC1): track 0.00 -> 10.2 mm
- net Net-(J2-CC2): track 0.00 -> 8.65 mm
- net +12V: track 0.00 -> 8.48 mm, vias 0 -> 2
- net Net-(F1-Pad1): track 0.00 -> 7.74 mm
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- added copper zone on F.Cu, net (none)
- added copper zone on In2.Cu, net +12V
- added copper zone on F.Cu, net +24V
- added copper zone on In2.Cu, net +24V
- added copper zone on In2.Cu, net +3.3V
- added copper zone on F.Cu, net /SW
- added copper zone on F.Cu, net AGND
- added copper zone on F.Cu, net PGND
Other:
- rule pad_to_mask_clearance: 0 -> 0.0508
