File: BreadBoard_git/BreadBoard_git.kicad_pcb (KiCad board)
At the start: 4 copper layers, 119 x 62.6 mm, 88 parts, among them J1 PD-40, J2 USB_C_Receptacle_USB2.0_14P, J4 Conn_01x02_Pin, J5 Conn_01x02_Pin, J7 Conn_01x15_Pin, J8 Conn_01x05_Pin, Q1 CSD18512Q5B, Q3 CSD18512Q5B, Q5 RQ3E110AJTB, Q6 RQ3E110AJTB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

Commit message: updates!
Parts:
- moved J2 43.6 mm to (170.4, 53.6), turned to 180 degrees
- moved R6 43.2 mm to (163.3, 54.2), turned to 90 degrees
- moved R4 43.0 mm to (161.8, 54.7), turned to 90 degrees
- moved C8 36.6 mm to (177.1, 59.3), turned to 0 degrees
- moved Cin8 36.3 mm to (79.0, 86.0)
- moved C7 34.5 mm to (177.1, 60.5), turned to 0 degrees
- moved D2 32.7 mm to (160.6, 58.5)
- moved D5 29.8 mm to (171.5, 60.8), turned to 90 degrees
- moved D6 29.7 mm to (166.3, 60.5), turned to 90 degrees
- moved D4 29.2 mm to (169.7, 60.8), turned to 90 degrees
- moved R2 21.2 mm to (154.7, 89.5), turned to 90 degrees
- moved C5 21.1 mm to (155.1, 83.1), turned to -90 degrees
- moved R18 20.8 mm to (144.8, 63.8)
- moved C2 20.8 mm to (146.8, 63.9)
- moved U4 20.8 mm to (154.2, 64.8)
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Connections:
- Cout1 pad 2: GND -> PGND
- Cout2 pad 2: GND -> PGND
- Cout3 pad 2: GND -> PGND
- Cout9 pad 2: GND -> PGND
- D1 pad A: GND -> PGND
- J1 pad 2: GND -> PGND
- J1 pad 3: GND -> PGND
- J1 pad S1: GND -> PGND
- SW1 pad 2: unconnected-(SW1-Pad2) -> /CHIP_PU
- SW1 pad 4: unconnected-(SW1-Pad4) -> GND
- SW2 pad 2: unconnected-(SW2-Pad2) -> /BOOT
- SW2 pad 4: unconnected-(SW2-Pad4) -> GND
- TP4 pad 1: GND -> PGND
Routing:
- net PGND: track 0.10 -> 121.8 mm, vias 0 -> 2
- net /ISNS_P: track 0.00 -> 43.7 mm, vias 0 -> 2
- net /CHIP_PU: track 6.22 -> 47.8 mm, vias 0 -> 2
- net /BOOT: track 0.00 -> 27.8 mm, vias 0 -> 2
- net /USB_D-: track 54.2 -> 27.5 mm
- net /USB_D+: track 55.0 -> 28.5 mm
- net GND: track 25.4 -> 50.2 mm, vias 20 -> 40
- net /SDA: track 20.6 -> 0.03 mm
- net /SCL: track 20.5 -> 0.03 mm
- net +24V: track 13.0 -> 30.6 mm, vias 11 -> 13
- net +3.3V: track 2.96 -> 19.5 mm, vias 2 -> 7
- net /HO: track 0.00 -> 15.9 mm, vias 0 -> 2
- net /LO: track 0.00 -> 15.2 mm, vias 0 -> 2
- net Net-(U2-EN/SYNC): track 0.00 -> 12.3 mm
- net +5V: track 0.00 -> 11.6 mm, vias 0 -> 1
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- added copper zone on In2.Cu, net +5V
- added copper zone on In2.Cu, net +5V_IN
- added copper zone on In2.Cu, net +5V_USB
Other:
- board size 119 x 62.6 mm -> 117.4 x 54 mm

Commit message: updates
Parts:
- removed TP1: 24V_in, TestPoint:TestPoint_Keystone_5019_Miniature
- removed TP2: +24_gnd, TestPoint:TestPoint_Keystone_5019_Miniature
- removed TP3: 12V_out, TestPoint:TestPoint_Keystone_5019_Miniature
- removed TP4: gnd, TestPoint:TestPoint_Keystone_5019_Miniature
- removed TP5: 5out, TestPoint:TestPoint_Keystone_5019_Miniature
- removed TP6: 5v_out, TestPoint:TestPoint_Keystone_5019_Miniature
- removed TP7: 3.3V, TestPoint:TestPoint_Keystone_5019_Miniature
- added Cinblk2: 10uF, Capacitor_SMD:C_1210_3225Metric_Pad1.33x2.70mm_HandSolder, F.Cu at (114.6, 57.2)
- added G***: LOGO, footprints:bread, F.Cu at (87.9, 97.5)
- added J6: Conn_01x08_Socket, Connector_PinSocket_2.54mm:PinSocket_1x08_P2.54mm_Vertical, F.Cu at (157.9, 102.2)
- moved R26 53.5 mm to (166.2, 97.6), turned to 180 degrees
- moved R25 52.6 mm to (168.9, 98.6), turned to -90 degrees
- moved R28 52.3 mm to (135.6, 92.0), turned to 180 degrees
- moved R27 51.3 mm to (145.1, 92.0), turned to 180 degrees
- moved J5 47.3 mm to (130.6, 101.5), turned to 90 degrees
- moved Q6 47.2 mm to (145.1, 95.5), turned to -90 degrees
- moved J4 46.1 mm to (140.5, 101.5), turned to 90 degrees
- moved Q5 43.1 mm to (135.7, 95.3), turned to -90 degrees
- moved Cin8 32.8 mm to (109.1, 98.9)
- moved J8 28.6 mm to (165.1, 69.7), turned to 0 degrees
- moved SW1 25.9 mm to (172.4, 67.3), turned to 0 degrees
- moved R1 23.2 mm to (168.6, 70.9), turned to 0 degrees
- moved C5 21.6 mm to (172.8, 70.9), turned to 0 degrees
- moved SW2 21.0 mm to (154.3, 68.5), turned to 0 degrees
- moved C6 18.5 mm to (155.5, 71.3), turned to 0 degrees
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Connections:
- net /HO renamed /SW-
- net /SW renamed /SW+
- net Net-(F1-Pad1) renamed /vbus
- J4 pad 1: /Heater1- -> +12V
- J5 pad 2: +12V -> /Heater1-
- R25 pad 1: /GPIO6 -> /GPIO41
- R26 pad 1: /GPIO7 -> /GPIO40
- U5 pad 12: /MOSI -> unconnected-(U5-IO8-Pad12)
- U5 pad 18: /CS -> /MISO
- U5 pad 19: /MISO -> /MOSI
- U5 pad 20: /RST -> /CS
- U5 pad 21: /DINT -> /RST
- U5 pad 22: unconnected-(U5-IO14-Pad22) -> /DINT
- U5 pad 31: unconnected-(U5-IO38-Pad31) -> /GPIO38
- U5 pad 32: unconnected-(U5-IO39-Pad32) -> /GPIO39
- U5 pad 33: unconnected-(U5-IO40-Pad33) -> /GPIO40
- U5 pad 34: unconnected-(U5-IO41-Pad34) -> /GPIO41
- U5 pad 35: unconnected-(U5-IO42-Pad35) -> /GPIO42
- U5 pad 36: unconnected-(U5-RXD0-Pad36) -> /RXDO
- U5 pad 37: unconnected-(U5-TXD0-Pad37) -> /TXD0
- U5 pad 38: unconnected-(U5-IO2-Pad38) -> /GPIO2
- U5 pad 39: unconnected-(U5-IO1-Pad39) -> /GPIO1
- U5 pad 6: /GPIO6 -> unconnected-(U5-IO6-Pad6)
- U5 pad 7: /GPIO7 -> unconnected-(U5-IO7-Pad7)
Routing:
- net PGND: track 121.8 -> 25.8 mm, vias 2 -> 27
- net Net-(Q5-Pad4): track 0.00 -> 38.2 mm
- net Net-(Q6-Pad4): track 0.00 -> 32.3 mm
- net /CHIP_PU: track 47.8 -> 18.3 mm, vias 2 -> 0
- net +12V: track 13.2 -> 41.9 mm, vias 1 -> 5
- net +24V: track 30.6 -> 4.19 mm, vias 13 -> 21
- net /GPIO42: track 0.00 -> 11.5 mm, vias 0 -> 1
- net /GPIO38: track 0.00 -> 10.7 mm, vias 0 -> 1
- net /CS: track 14.4 -> 3.87 mm, vias 2 -> 0
- net /RXDO: track 0.00 -> 10.1 mm
- net /MOSI: track 14.1 -> 4.20 mm, vias 2 -> 0
- net /GPIO39: track 0.00 -> 9.88 mm, vias 0 -> 1
- net /BOOT: track 27.8 -> 37.1 mm
- net /TXD0: track 0.00 -> 8.42 mm
- net /VDDA: track 4.37 -> 12.7 mm, vias 0 -> 2
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- added copper zone on F.Cu, net +3.3V
- added copper zone on F.Cu, net +5V_IN
- added copper zone on F.Cu, net /Heater1-
- added copper zone on F.Cu, net /Heater2-
- added copper zone on F.Cu, net /vbus
- added copper zone on F.Cu, net GND
- added copper zone on In1.Cu, net PGND
Other:
- board size 117.4 x 54 mm -> 107.8 x 53.6 mm
- board text added: "12V"
- board text added: "5V Selection"
- board text added: "5V USB"
- board text added: "5V Wall"
- board text added: "DISPLAY"
- board text added: "GND"
- board text added: "HEATER 1"
- board text added: "HEATER 2"
- board text added: "Natalie Cooper & Mary Newell Breadboard"
- board text added: "SCL SDA x GND 3.3V"
- board text added: "TEMP/HUMIDITY"
- board text added: "x x x x DINT X RST CS MOSI MISO SCK X X GND 3.3V"
